File: boards/2018_Example_Project/2018_Example_Project.kicad_pcb (KiCad board)
At the start: 2 copper layers, 37 parts, among them J1 Mounting_Hole_4-40, J2 Mounting_Hole_4-40, J3 Mounting_Hole_4-40, J4 Mounting_Hole_4-40, J5 Ultrafit_4, Q1 NMOS_GSD_30V, Q2 NMOS_GSD_30V, U1 TPS561201, U2 MCP603

Commit message: added board dxf
Other:
- board outline added: 70 x 70 mm
Changed lines of the file:
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@@
     (links 54)
     (no_connects 54)
-    (area 0 0 0 0)
+    (area 120.037619 86.275 187.929524 125.895)
     (thickness 1.6)
-    (drawings 0)
+    (drawings 12)
     (tracks 0)
     (zones 0)
@@
     )
   )
+  (gr_arc (start 186.07 140.23) (end 186.07 142.77) (angle -90) (layer Edge.Cuts) (width 0.1))
+  (gr_arc (start 186.07 75.31) (end 188.61 75.31) (angle -90) (layer Edge.Cuts) (width 0.1))
+  (gr_arc (start 121.15 75.31) (end 121.15 72.77) (angle -90) (layer Edge.Cuts) (width 0.1))
+  (gr_arc (start 121.15 140.23) (end 118.61 140.23) (angle -90) (layer Edge.Cuts) (width 0.1))
+  (gr_line (start 121.15 142.77) (end 186.07 142.77) (layer Edge.Cuts) (width 0.1))
+  (gr_line (start 188.61 140.23) (end 188.61 75.31) (layer Edge.Cuts) (width 0.1))
+  (gr_line (start 186.07 72.77) (end 121.15 72.77) (layer Edge.Cuts) (width 0.1))
+  (gr_line (start 118.61 75.31) (end 118.61 140.23) (layer Edge.Cuts) (width 0.1))
+  (gr_circle (center 124.96 79.171941) (end 126.59195 79.171941) (layer Edge.Cuts) (width 0.1))
+  (gr_circle (center 124.96 136.368059) (end 126.59195 136.368059) (layer Edge.Cuts) (width 0.1))
+  (gr_circle (center 182.26 136.368059) (end 183.89195 136.368059) (layer Edge.Cuts) (width 0.1))
+  (gr_circle (center 182.26 79.171941) (end 183.89195 79.171941) (layer Edge.Cuts) (width 0.1))
 )
