File: boards/dashboard/dashboard.sch (KiCad schematic (older format))
At the start: 32 parts

Commit message: Fixed dashboard schematic, added CP2120 breakout Gerber files
Parts:
- removed J?: micromatch_male_10, symbol micromatch_male_10
- added C10: 10uF, Capacitors_SMD:C_0805, symbol C_47uF
- added C9: 0.1uF, Capacitors_SMD:C_0805, symbol C_47uF
- added D1: D_Zener_18V, footprints:DO-214AA, symbol D_Zener_18V
- added J1: micromatch_male_10, symbol micromatch_male_10
- added R11, R13, R14: 4.7k, symbol R
- added U3: LM1117-3.3, symbol LM1117-3.3
- gave numbers to parts that had none: 31
Connections:
- net +12V: now also D1.1 (K)
- net AMS: now also J1.6
- net GND: now also U4.GND, C10.2, C9.2, D1.2 (A), J1.3, J1.5, J1.7, U3.1 (GND)
- net IMD: now also J1.4
- net SCL: now also J1.10, R13.2
- net SDA: now also J1.9, R14.2
- net START: now also J1.2
- net VCC: now also C9.1, J1.1, J1.8, U3.3 (VI); no longer U4.3 (VDD)
- net at C3.1, F1.2, R1.1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: now also U2.3 (VIN)
- net at R3.2, U2.5 (EN): no longer U2.3 (VIN)
- net at U4.4 (RST): now also R11.2
- net RESET renamed AT_RESET
- new net +3V3: C10.1, R11.1, R13.1, R14.1, U3.2 (VO), U4.3 (VDD)
- no-connect marks 1 -> 27
Other:
- moved on the sheet: J2, Q1, R12, U4

Commit message: Revisions to CP2120 board files
Parts:
- added C11: 0.1uF, Capacitors_SMD:C_0805, symbol C_47uF
- J1: footprint (none) -> footprints:micromatch_female_ra_10
- J2: footprint (none) -> footprints:micromatch_female_ra_14
- R11, R12, R13, R14, R8, R9: footprint (none) -> footprints:R_0805_OEM
- U3: footprint (none) -> SparkFun-PowerIC:SOT223
- U4: footprint (none) -> footprints:CP2120-QFN
Connections:
- net +3V3: now also C11.1; no longer R11.1
- net GND: now also C11.2; no longer C10.2
Other:
- moved on the sheet: C10, C9, Q1, R12, U3
