File: boards/IMD_Latch/IMD_Latch.kicad_pcb (KiCad board)
At the start: 2 copper layers, 0 parts

Commit message: Starting Layout
Parts:
- added C1: C_10uF, footprints:C_0805_OEM, F.Cu at (171.4, 66.0)
- added C2: C_22uF, footprints:C_1206_OEM, F.Cu at (171.4, 119.4)
- added C3: C_0.1uF, footprints:C_0805_OEM, F.Cu at (178.8, 113.3)
- added C4: C_47uF, footprints:C_0805_OEM, F.Cu at (171.4, 72.4)
- added D1: LED_0805, footprints:LED_0805_OEM, F.Cu at (171.4, 114.3)
- added D2: LED_0805, footprints:LED_0805_OEM, F.Cu at (116.8, 79.4)
- added D3: D_Zener_18V, footprints:DO-214AA, F.Cu at (159.4, 118.1)
- added D4: D_Schottky_SOD123, footprints:D_SOD-123W_OEM, F.Cu at (121.9, 81.9)
- added D5: D_Schottky_SOD123, footprints:D_SOD-123W_OEM, F.Cu at (111.8, 81.9)
- added D6: D_Schottky_SOD123, footprints:D_SOD-123W_OEM, F.Cu at (111.1, 91.4)
- added D7: LED_0805, footprints:LED_0805_OEM, F.Cu at (120.7, 91.4)
- added F1: F_500mA_16V, footprints:Fuse_1210, F.Cu at (168.3, 118.1)
- added J1: micromatch_female_RA_8, footprints:micromatch_female_ra_8, F.Cu at (151.8, 128.3)
- added J2: Ultrafit_2, footprints:Ultrafit_2, F.Cu at (135.3, 102.2)
- added K1: G5Q-1A4-DC5-5V, footprints:Relay_SPST_OMRON-G5Q-1A4_OEM, F.Cu at (167.6, 96.5)
- added L1: L_4.7uH, footprints:4.7uH_Inductor_OEM, F.Cu at (133.3, 114.9)
- added Q1: SSM3K333R, footprints:SOT-23F, F.Cu at (134.6, 124.5)
- added R1: R_402k, footprints:R_0805_OEM, F.Cu at (197.5, 79.4)
- added R10: R_200, footprints:R_0805_OEM, F.Cu at (197.5, 93.3)
- added R11: R_200, footprints:R_0805_OEM, F.Cu at (208.3, 97.8)
- added R12: R_1k, footprints:R_0805_OEM, F.Cu at (202.6, 79.4)
- added R2: R_1k, footprints:R_0805_OEM, F.Cu at (174.6, 114.3)
- added R3: R_1.07k, footprints:R_0805_OEM, F.Cu at (201.3, 86.4)
- added R4: R_402k, footprints:R_0805_OEM, F.Cu at (205.1, 84.5)
- added R5: R_10k, footprints:R_0805_OEM, F.Cu at (174.6, 118.1)
- added R6: R_10k, footprints:R_0805_OEM, F.Cu at (201.9, 99.7)
- added R7: R_55.1k, footprints:R_0805_OEM, F.Cu at (205.7, 93.3)
- added R8: R_0_Jumper, footprints:R_2512_OEM, F.Cu at (193.7, 83.8)
- added R9: R_1.13k, footprints:R_0805_OEM, F.Cu at (196.2, 99.7)
- added U1: TPS561201, footprints:SOT-23-6_OEM, F.Cu at (178.8, 116.3)
- added U2: TLP175A_OEM, footprints:SOIC-8_3.9x4.9mm_Pitch1.27mm_OEM, F.Cu at (153.0, 84.5)
- added U3: TS507IYLT, footprints:SOT-23-5_OEM, F.Cu at (159.4, 90.8)

Commit message: Layout01
Parts:
- U2: footprint footprints:SOIC-8_3.9x4.9mm_Pitch1.27mm_OEM -> footprints:MFSOP6-4_4.4x3.6mm_Pitch1.27mm_OEM
- moved R11 70.3 mm to (138.8, 108.7), turned to 90 degrees
- moved R3 63.4 mm to (139.0, 98.1), turned to 270 degrees
- moved D4 58.8 mm to (167.8, 118.6), turned to 90 degrees
- moved D5 57.1 mm to (154.9, 119.4)
- moved D2 53.4 mm to (163.8, 104.7)
- moved R4 52.8 mm to (164.6, 118.3), turned to 90 degrees
- moved R12 52.0 mm to (163.0, 113.1), turned to 90 degrees
- moved C1 47.3 mm to (166.0, 113.1), turned to 270 degrees
- moved R1 44.2 mm to (168.8, 113.0), turned to 270 degrees
- moved R9 42.8 mm to (154.4, 109.0), turned to 180 degrees
- moved R7 41.2 mm to (164.9, 98.6), turned to 90 degrees
- moved R6 39.8 mm to (162.2, 98.7), turned to 90 degrees
- moved L1 39.0 mm to (165.1, 92.2)
- moved J1 37.5 mm to (132.2, 96.3)
- moved R10 37.1 mm to (163.9, 109.2), turned to 180 degrees
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Connections:
- D5 pad 1: Net-(D4-Pad1) -> Net-(D5-Pad1)
- D5 pad 2: Net-(D5-Pad2) -> Net-(D4-Pad1)
- D6 pad 1: Net-(D5-Pad2) -> Net-(D5-Pad1)
- K1 pad 5: Net-(D5-Pad2) -> Net-(D5-Pad1)
- U2 pad 4: Net-(D5-Pad2) -> Net-(D5-Pad1)
Routing:
- net Net-(D5-Pad1): track 0.00 -> 0.85 mm
Other:
- net class Default: trace_width 0.1524 -> 0.254
- board text added: "12V LED"
- board text added: "2017-18"
- board text added: "5V LED"
- board text added: "Buck Converter"
- board text added: "IMD Latch"
- board text added: "Josh Deng"
- board text added: "Motorsports"
- board text added: "Olin Electric"
- board text added: "Op-amp LED"

Commit message: Layout finished
Parts:
- moved D5 0.75 mm to (154.4, 118.8)
- moved D2 0.74 mm to (163.4, 104.1), turned to 270 degrees
- moved U1 0.67 mm to (157.1, 95.5)
- moved D6 0.67 mm to (143.9, 98.2)
- moved U3 0.46 mm to (154.2, 114.0)
- moved R3 0.40 mm to (138.6, 98.2), turned to 0 degrees
- moved R7 0.37 mm to (165.2, 98.8)
- moved D7 0.35 mm to (138.6, 102.9)
- moved C4 0.20 mm to (168.7, 98.8), turned to 270 degrees
- moved Q1 0.19 mm to (160.4, 119.0)
- moved R6 0.17 mm to (162.1, 98.6), turned to 270 degrees
- moved D1 0.06 mm to (149.0, 89.9), turned to 90 degrees
- turned R2 to 90 degrees
Routing:
- net Net-(D5-Pad1): track 0.85 -> 0.00 mm
Other:
- board text added: "IMD Latch v1"
- board text removed: "IMD Latch"

Commit message: Tracing ready Layout
Parts:
- moved U3 21.4 mm to (134.7, 105.0)
- moved R9 19.2 mm to (137.9, 99.1)
- moved J2 17.2 mm to (151.1, 115.7), turned to 90 degrees
- moved C4 15.0 mm to (153.7, 98.6), turned to 180 degrees
- moved D4 14.2 mm to (156.2, 110.3), turned to 0 degrees
- moved D5 12.4 mm to (154.9, 106.4), turned to 90 degrees
- moved D7 12.3 mm to (135.8, 114.9), turned to 90 degrees
- moved R1 12.2 mm to (158.2, 107.0)
- moved R6 11.9 mm to (150.5, 101.5), turned to 90 degrees
- moved D1 11.6 mm to (137.4, 89.5), turned to 0 degrees
- moved L1 11.3 mm to (153.7, 92.1)
- moved R7 11.3 mm to (154.3, 101.6)
- moved C3 11.1 mm to (146.1, 89.7)
- moved R2 10.7 mm to (142.0, 89.7), turned to 180 degrees
- moved U1 9.91 mm to (147.2, 94.3)
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Connections:
- D5 pad 1: Net-(D5-Pad1) -> Net-(D4-Pad1)
- D5 pad 2: Net-(D4-Pad1) -> Net-(D5-Pad2)
- D6 pad 1: Net-(D5-Pad1) -> Net-(D5-Pad2)
- K1 pad 5: Net-(D5-Pad1) -> Net-(D5-Pad2)
- U2 pad 4: Net-(D5-Pad1) -> Net-(D5-Pad2)
Routing:
- net Net-(J2-Pad1): track 0.00 -> 17.0 mm
- net Net-(J2-Pad2): track 0.00 -> 13.6 mm
Other:
- board text removed: "Buck Converter"
- board text removed: "Motorsports"
- board text removed: "Olin Electric"

Commit message: IMD Latch Tracing for the first time
Parts:
- moved R2 0.16 mm to (142.1, 89.5)
Routing:
- net GND: track 0.00 -> 58.2 mm, vias 0 -> 3
- net VCC: track 0.00 -> 40.9 mm, vias 0 -> 2
- net /12V_Fused: track 0.00 -> 35.6 mm, vias 0 -> 2
- net Net-(C4-Pad1): track 0.00 -> 25.7 mm
- net Net-(R11-Pad1): track 0.00 -> 19.1 mm
- net Net-(R12-Pad1): track 0.00 -> 18.2 mm, vias 0 -> 2
- net Net-(D4-Pad1): track 0.11 -> 16.3 mm
- net Net-(C3-Pad2): track 0.00 -> 14.9 mm
- net Net-(D5-Pad2): track 0.00 -> 13.5 mm
- net Net-(R6-Pad1): track 0.00 -> 12.1 mm
- net +12V: track 0.00 -> 12.1 mm
- net Net-(R3-Pad2): track 0.00 -> 9.71 mm
- net Net-(Q1-Pad3): track 0.00 -> 8.68 mm
- net Net-(C1-Pad1): track 0.12 -> 7.49 mm
- net Net-(J1-Pad3): track 0.00 -> 7.30 mm
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- added copper zone on B.Cu, net GND

Commit message: preparing for v2
Parts:
- removed D4, D5: D_Schottky_SOD123, footprints:D_SOD-123W_OEM
- moved U2 1.83 mm to (152.3, 107.8)
Connections:
- Q1 pad 1: Net-(D4-Pad1) -> Net-(C1-Pad1)
- R4 pad 1: Net-(D4-Pad1) -> Net-(C1-Pad1)
Routing:
- net GND: track 58.2 -> 32.5 mm, vias 3 -> 6
- net VCC: track 40.9 -> 15.4 mm, vias 2 -> 0
- net Net-(D4-Pad1): track 16.3 -> 0.00 mm
- net Net-(C1-Pad1): track 7.49 -> 13.4 mm
- net Net-(R11-Pad1): track 19.1 -> 22.2 mm
- net Net-(Q1-Pad3): track 8.68 -> 6.23 mm
- net Net-(D6-Pad1): track 13.5 -> 11.8 mm
- net Net-(R12-Pad1): track 18.2 -> 17.4 mm
