File: boards/IMD_Latch/IMD_Latch.sch (KiCad schematic (older format))
At the start: 43 parts

Commit message: Redesigned IMD Latch
Parts:
- removed C?: C_1uF, Capacitors_SMD:C_0805, symbol C_1uF
- removed C?: C_10uF, Capacitors_SMD:C_0805, symbol C_10uF
- removed C?: C_0.1uF, Capacitors_SMD:C_0805, symbol C_0.1uF
- removed C?: C_0.33uF, Capacitors_SMD:C_0805, symbol C_0.33uF
- removed D? (x2): LED_0805, LEDs:LED_0805, symbol LED_0805
- removed D? (x3): D_Schottky_SOD123, Diodes_SMD:D_SOD-123, symbol D_Schottky_SOD123
- removed F?: F_500mA_16V, footprints:Fuse_1210, symbol F_500mA_16V
- removed J?: micromatch_male_8, symbol micromatch_male_8
- removed J?: Ultrafit_4, footprints:Ultrafit_4, symbol Ultrafit_4
- removed K?: G6C-1117P-US, footprints:Relay_SPST_OMRON-G6C, symbol G6C-1117P-US
- removed Q?: LM78L05ACZ_Voltage_Regulator, footprints:TO-92-3_Inline_Narrow_Oval, symbol LM78L05ACZ_Voltage_Regulator
- removed Q? (x3): SSM3K333R, footprints:SOT-23F, symbol SSM3K333R
- removed R? (x2): R_200, Resistors_SMD:R_0805, symbol R_200
- removed R?: R_200k, Resistors_SMD:R_0805, symbol R_200k
- removed R?: R_22M, Resistors_SMD:R_0805, symbol R_22M
- removed R?: R_1M, Resistors_SMD:R_0805, symbol R_1M
- removed R? (x3): R_100k, Resistors_SMD:R_0805, symbol R_100k
- removed R?: R_2.2k, Resistors_SMD:R_0805, symbol R_2.2k
- removed U?: LMV341, TO_SOT_Packages_SMD:SOT-23-6, symbol LMV341
- removed U?: SN74LVC1G123DCTR, symbol SN74LVC1G123DCTR
- removed U?: TLP175A, Housings_SSOP:MFSOP6-4_4.4x3.6mm_Pitch1.27mm, symbol TLP175A
- added C1: C_10uF, footprints:C_0805_OEM, symbol C_10uF
- added D3: D_Zener_18V, footprints:DO-214AA, symbol D_Zener_18V
- added D4, D5, D6: D_Schottky_SOD123, footprints:D_SOD-123W_OEM, symbol D_Schottky_SOD123
- added D7: LED_0805, footprints:LED_0805_OEM, symbol LED_0805
- added F1: F_500mA_16V, footprints:Fuse_1210, symbol F_500mA_16V
- added J1: micromatch_female_RA_8, footprints:micromatch_female_ra_8, symbol micromatch_female_RA_8
- added J2: Ultrafit_2, footprints:Ultrafit_2, symbol Ultrafit_2
- added K1: G5Q-1A4-DC5-5V, footprints:Relay_SPST_OMRON-G5Q-1A4_OEM, symbol G5Q-1A4-DC5-5V
- added Q1: SSM3K333R, footprints:SOT-23F, symbol SSM3K333R
- added R1, R4: R_402k, footprints:R_0805_OEM, symbol R_402k
- added R11: R_200, footprints:R_0805_OEM, symbol R_200
- added R3: R_1.07k, Resistors_SMD:R_0805, symbol R_1.07k
- added R9: R_1.13k, Resistors_SMD:R_0805, symbol R_1.13k
- added U2: TLP175A_OEM, footprints:SOIC-8_3.9x4.9mm_Pitch1.27mm_OEM, symbol TLP175A_OEM
- added U3: TS507IYLT, footprints:SOT-23-5_OEM, symbol TS507IYLT
- gave numbers to parts that had none: 14
Connections:
- net +12V: now also D3.2 (A), F1.1, J1.2
- net 12V_Fused: now also U1.3 (VIN), F1.2, J1.5
- net GND: now also C1.2, D3.1 (K), D6.2 (A), D7.1 (K), J1.1, J1.4, J1.6, J1.7, K1.1, Q1.2 (S), R4.2, R9.1, U3.2 (V-)
- net VCC: now also R1.1, U3.5 (V+)
- net at R5.2, U1.5 (EN): no longer U1.3 (VIN)
- net at R12.1: now also U2.1
- new net: J1.3, R3.1
- new net: J2.1, K1.2
- new net: J2.2, K1.3
- new net: D5.2 (A), D6.1 (K), K1.5, U2.4
- new net: R3.2, R9.2, U3.1 (+)
- new net: R11.1, U2.6, U3.3 (-), U3.4
- new net: Q1.3 (D), U2.3
- new net: D7.2 (A), R11.2
- new net: D4.1 (K), D5.1 (K), Q1.1 (G), R4.1
- new net: C1.1, D4.2 (A), R1.2
- no-connect marks 0 -> 1
Other:
- note removed: "IMD Latch"
- note removed: "IMD Status\n"
- moved on the sheet: C2, C3, C4, D1, D2, L1, R10, R12, R2, R5, R6, R7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

Commit message: Layout Ready IMD Latch
Parts:
- C2: footprint Capacitors_SMD:C_1206 -> footprints:C_1206_OEM
- C3, C4: footprint Capacitors_SMD:C_0805 -> footprints:C_0805_OEM
- D1, D2: footprint LEDs:LED_0805 -> footprints:LED_0805_OEM
- R10, R12, R2, R3, R5, R6, R7, R9: footprint Resistors_SMD:R_0805 -> footprints:R_0805_OEM
- R8: footprint Resistors_SMD:R_2512 -> footprints:R_2512_OEM
- U1: footprint TO_SOT_Packages_SMD:SOT-23-6 -> footprints:SOT-23-6_OEM
Connections:
- net +12V: now also D3.1 (K); no longer D3.2 (A)
- net GND: now also D3.2 (A); no longer D3.1 (K)
Changed lines of the file:
@@
 F 0 "R5" V 2180 2250 50  0000 C CNN
 F 1 "R_10k" V 2000 2250 50  0000 C CNN
-F 2 "Resistors_SMD:R_0805" H 2030 2250 50  0001 C CNN
+F 2 "footprints:R_0805_OEM" H 2030 2250 50  0001 C CNN
 F 3 "http://www.bourns.com/data/global/pdfs/CRS.pdf" H 2180 2250 50  0001 C CNN
 F 4 "CRS0805-FX-1002ELFCT-ND" H 2100 2250 60  0001 C CNN "MPN"
@@
 F 0 "R6" V 3230 2400 50  0000 C CNN
 F 1 "R_10k" V 3050 2400 50  0000 C CNN
-F 2 "Resistors_SMD:R_0805" H 3080 2400 50  0001 C CNN
+F 2 "footprints:R_0805_OEM" H 3080 2400 50  0001 C CNN
 F 3 "http://www.bourns.com/data/global/pdfs/CRS.pdf" H 3230 2400 50  0001 C CNN
 F 4 "CRS0805-FX-1002ELFCT-ND" H 3150 2400 60  0001 C CNN "MPN"
@@
 F 0 "R2" V 1680 2400 50  0000 C CNN
 F 1 "R_1k" V 1500 2400 50  0000 C CNN
-F 2 "Resistors_SMD:R_0805" H 1530 2400 50  0001 C CNN
+F 2 "footprints:R_0805_OEM" H 1530 2400 50  0001 C CNN
 F 3 "https://www.seielect.com/Catalog/SEI-rncp.pdf" H 1680 2400 50  0001 C CNN
 F 4 "Digi-Key" H 1600 2400 60  0001 C CNN "MFN"
@@
 F 0 "R7" V 3250 2250 50  0000 C CNN
 F 1 "R_55.1k" V 3450 2250 50  0000 C CNN
-F 2 "Resistors_SMD:R_0805" H 3280 2250 50  0001 C CNN
+F 2 "footprints:R_0805_OEM" H 3280 2250 50  0001 C CNN
 F 3 "http://www.yageo.com.tw/exep/pages/download/literatures/PYu-R_INT-thick_7.pdf" H 3430 2250 50  0001 C CNN
 F 4 "311-51.1KCRCT-ND" H 3350 2250 60  0001 C CNN "MPN"
@@
 F 0 "R10" V 4300 2200 50  0000 C CNN
 F 1 "R_200" V 4500 2200 50  0000 C CNN
-F 2 "Resistors_SMD:R_0805" H 4330 2200 50  0001 C CNN
+F 2 "footprints:R_0805_OEM" H 4330 2200 50  0001 C CNN
 F 3 "https://www.seielect.com/Catalog/SEI-RMCF_RMCP.pdf" H 4480 2200 50  0001 C CNN
 F 4 "Digi-Key" H 4400 2200 60  0001 C CNN "MFN"
@@
 F 0 "R8" V 4130 2050 50  0000 C CNN
 F 1 "R_0_Jumper" V 3950 2050 50  0000 C CNN
-F 2 "Resistors_SMD:R_2512" H 3980 2050 50  0001 C CNN
+F 2 "footprints:R_2512_OEM" H 3980 2050 50  0001 C CNN
 F 3 "http://www.te.com/commerce/DocumentDelivery/DDEController?Action=srchrtrv&DocNm=9-1773463-7&DocType=DS&DocLang=English" H 4130 2050 50  0001 C CNN
 F 4 "A121322CT-ND" H 4050 2050 60  0001 C CNN "MPN"
@@
 F 0 "D1" H 1600 2600 50  0000 C CNN
 F 1 "LED_0805" H 1600 2800 50  0000 C CNN
-F 2 "LEDs:LED_0805" H 1500 2700 50  0001 C CNN
+F 2 "footprints:LED_0805_OEM" H 1500 2700 50  0001 C CNN
 F 3 "http://www.osram-os.com/Graphics/XPic9/00078860_0.pdf" H 1600 2800 50  0001 C CNN
 F 4 "475-1410-1-ND" H 1600 2700 60  0001 C CNN "MPN"
@@
 F 0 "D2" H 4400 2400 50  0000 C CNN
 F 1 "LED_0805" H 4400 2600 50  0000 C CNN
-F 2 "LEDs:LED_0805" H 4300 2500 50  0001 C CNN
+F 2 "footprints:LED_0805_OEM" H 4300 2500 50  0001 C CNN
 F 3 "http://www.osram-os.com/Graphics/XPic9/00078860_0.pdf" H 4400 2600 50  0001 C CNN
 F 4 "475-1410-1-ND" H 4400 2500 60  0001 C CNN "MPN"
@@
 F 0 "C3" H 3350 1800 50  0000 L CNN
 F 1 "C_0.1uF" H 3350 2000 50  0000 L CNN
-F 2 "Capacitors_SMD:C_0805" H 3338 1750 50  0001 C CNN
+F 2 "footprints:C_0805_OEM" H 3338 1750 50  0001 C CNN
 F 3 "http://datasheets.avx.com/X7RDielectric.pdf" H 3325 2000 50  0001 C CNN
 F 4 "478-3352-1-ND" H 3300 1900 60  0001 C CNN "MPN"
@@
 F 0 "C2" H 1875 2500 50  0000 L CNN
 F 1 "C_22uF" H 1875 2300 50  0000 L CNN
-F 2 "Capacitors_SMD:C_1206" H 1888 2250 50  0001 C CNN
+F 2 "footprints:C_1206_OEM" H 1888 2250 50  0001 C CNN
 F 3 "http://www.samsungsem.com/kr/support/product-search/mlcc/__icsFiles/afieldfile/2017/07/28/S_CL31A226KOCLFNC.pdf" H 1875 2500 50  0001 C CNN
 F 4 "1276-2725-1-ND" H 1850 2400 60  0001 C CNN "MPN"
@@
 F 0 "C4" H 3925 2500 50  0000 L CNN
 F 1 "C_47uF" H 3925 2300 50  0000 L CNN
-F 2 "Capacitors_SMD:C_0805" H 3938 2250 50  0001 C CNN
+F 2 "footprints:C_0805_OEM" H 3938 2250 50  0001 C CNN
 F 3 "http://www.yuden.co.jp/productdata/catalog/en/mlcc_all_e.pdf" H 3925 2500 50  0001 C CNN
 F 4 "587-4280-1-ND" H 3900 2400 60  0001 C CNN "MPN"
@@
 F 0 "U1" H 2500 1850 60  0000 C CNN
 F 1 "TPS561201" H 2700 2500 60  0000 C CNN
-F 2 "TO_SOT_Packages_SMD:SOT-23-6" H 2400 2400 60  0001 C CNN
+F 2 "footprints:SOT-23-6_OEM" H 2400 2400 60  0001 C CNN
 F 3 "http://www.ti.com/lit/ds/symlink/tps561201.pdf" H 2500 2500 60  0001 C CNN
 F 4 "Digi-Key" H 2700 2150 60  0001 C CNN "MFN"
@@
 F 0 "R12" V 6980 2350 50  0000 C CNN
 F 1 "R_1k" V 6900 2350 50  0000 C CNN
-F 2 "Resistors_SMD:R_0805" H 6830 2350 50  0001 C CNN
+F 2 "footprints:R_0805_OEM" H 6830 2350 50  0001 C CNN
 F 3 "https://www.seielect.com/Catalog/SEI-rncp.pdf" H 6980 2350 50  0001 C CNN
 F 4 "Digi-Key" H 6900 2350 60  0001 C CNN "MFN"
@@
 F 0 "R9" V 7330 1750 50  0000 C CNN
 F 1 "R_1.13k" V 7150 1750 50  0000 C CNN
-F 2 "Resistors_SMD:R_0805" H 7180 1750 50  0001 C CNN
+F 2 "footprints:R_0805_OEM" H 7180 1750 50  0001 C CNN
 F 3 "https://industrial.panasonic.com/cdbs/www-data/pdf/RDM0000/AOA0000C307.pdf" H 7330 1750 50  0001 C CNN
 F 4 "Digi-Key" H 7250 1750 60  0001 C CNN "MFN"
@@
 F 0 "R3" V 7330 1350 50  0000 C CNN
 F 1 "R_1.07k" V 7150 1350 50  0000 C CNN
-F 2 "Resistors_SMD:R_0805" H 7180 1350 50  0001 C CNN
+F 2 "footprints:R_0805_OEM" H 7180 1350 50  0001 C CNN
 F 3 "https://industrial.panasonic.com/cdbs/www-data/pdf/RDM0000/AOA0000C307.pdf" H 7330 1350 50  0001 C CNN
 F 4 "Digi-Key" H 7250 1350 60  0001 C CNN "MFN"
@@
 F 7 "https://www.digikey.com/products/en?keywords=SMBJ5355B-TPMSCT-ND" H 1600 2600 60  0001 C CNN "PurchasingLink"
 	1    1200 2100
-	0    -1   -1   0
-$EndComp
-Wire Wire Line
+	0    1    1    0
+$EndComp
+Wire Wire Line

Commit message: Layout01
Parts:
- U2: footprint footprints:SOIC-8_3.9x4.9mm_Pitch1.27mm_OEM -> footprints:MFSOP6-4_4.4x3.6mm_Pitch1.27mm_OEM
Connections:
- net at D6.1 (K), K1.5, U2.4: now also D5.1 (K); no longer D5.2 (A)
- net at D4.1 (K), Q1.1 (G), R4.1: now also D5.2 (A); no longer D5.1 (K)
Changed lines of the file:
@@
-$EndComp
-$Comp
-L TLP175A_OEM U2
-U 1 1 59F2E1E7
-P 7500 2450
-F 0 "U2" H 7300 2645 50  0000 L CNN
-F 1 "TLP175A_OEM" H 7300 2250 50  0000 L CNN
-F 2 "footprints:SOIC-8_3.9x4.9mm_Pitch1.27mm_OEM" H 7500 2150 50  0001 C CIN
-F 3 "https://toshiba.semicon-storage.com/info/docget.jsp?did=13665&prodName=TLP175A" H 7450 2450 50  0001 L CNN
-F 4 "TLP175A(TPLECT-ND" H 7400 2745 60  0001 C CNN "MPN"
-F 5 "Digi-Key" H 7500 2845 60  0001 C CNN "MFN"
-F 6 "https://www.digikey.com/product-detail/en/toshiba-semiconductor-and-storage/TLP175A-TPLE/TLP175A-TPLECT-ND/4562904" H 7600 2945 60  0001 C CNN "PurchasingLink"
-	1    7500 2450
-	1    0    0    -1
 $EndComp
 $Comp
@@
 $EndComp
 $Comp
-L D_Schottky_SOD123 D4
-U 1 1 59F40E3F
-P 6350 2950
-F 0 "D4" H 6350 3050 50  0000 C CNN
-F 1 "D_Schottky_SOD123" H 6350 2850 50  0000 C CNN
-F 2 "footprints:D_SOD-123W_OEM" H 6250 2950 50  0001 C CNN
-F 3 "https://assets.nexperia.com/documents/data-sheet/PMEG10010ELR.pdf" H 6350 3050 50  0001 C CNN
-F 4 "1727-2394-1-ND" H 6450 3150 60  0001 C CNN "MPN"
-F 5 "Digi-Key" H 6550 3250 60  0001 C CNN "MFN"
-F 6 "https://www.digikey.com/product-detail/en/nexperia-usa-inc/PMEG10010ELRX/1727-2394-1-ND/5436140" H 6650 3350 60  0001 C CNN "PurchasingLink"
-	1    6350 2950
-	-1   0    0    1
-$EndComp
-$Comp
-L D_Schottky_SOD123 D5
-U 1 1 59F41203
-P 7200 3750
-F 0 "D5" H 7200 3850 50  0000 C CNN
-F 1 "D_Schottky_SOD123" H 7200 3650 50  0000 C CNN
-F 2 "footprints:D_SOD-123W_OEM" H 7100 3750 50  0001 C CNN
-F 3 "https://assets.nexperia.com/documents/data-sheet/PMEG10010ELR.pdf" H 7200 3850 50  0001 C CNN
-F 4 "1727-2394-1-ND" H 7300 3950 60  0001 C CNN "MPN"
-F 5 "Digi-Key" H 7400 4050 60  0001 C CNN "MFN"
-F 6 "https://www.digikey.com/product-detail/en/nexperia-usa-inc/PMEG10010ELRX/1727-2394-1-ND/5436140" H 7500 4150 60  0001 C CNN "PurchasingLink"
-	1    7200 3750
-	1    0    0    -1
-$EndComp
-$Comp
-L D_Schottky_SOD123 D6
-U 1 1 59F41307
-P 7400 4400
-F 0 "D6" H 7400 4500 50  0000 C CNN
-F 1 "D_Schottky_SOD123" H 7400 4300 50  0000 C CNN
-F 2 "footprints:D_SOD-123W_OEM" H 7300 4400 50  0001 C CNN
-F 3 "https://assets.nexperia.com/documents/data-sheet/PMEG10010ELR.pdf" H 7400 4500 50  0001 C CNN
-F 4 "1727-2394-1-ND" H 7500 4600 60  0001 C CNN "MPN"
-F 5 "Digi-Key" H 7600 4700 60  0001 C CNN "MFN"
-F 6 "https://www.digikey.com/product-detail/en/nexperia-usa-inc/PMEG10010ELRX/1727-2394-1-ND/5436140" H 7700 4800 60  0001 C CNN "PurchasingLink"
-	1    7400 4400
-	0    1    1    0
-$EndComp
-$Comp
 L R_402k R1
 U 1 1 59F4430C
@@
 	1    0    0    -1
 $EndComp
+$Comp
+L TLP175A_OEM U2
+U 1 1 59F822D1
+P 7500 2450
+F 0 "U2" H 7300 2645 50  0000 L CNN
+F 1 "TLP175A_OEM" H 7300 2250 50  0000 L CNN
+F 2 "footprints:MFSOP6-4_4.4x3.6mm_Pitch1.27mm_OEM" H 7500 2150 50  0001 C CIN
+F 3 "https://toshiba.semicon-storage.com/info/docget.jsp?did=13665&prodName=TLP175A" H 7450 2450 50  0001 L CNN
+F 4 "TLP175A(TPLECT-ND" H 7400 2745 60  0001 C CNN "MPN"
+F 5 "Digi-Key" H 7500 2845 60  0001 C CNN "MFN"
+F 6 "https://www.digikey.com/product-detail/en/toshiba-semiconductor-and-storage/TLP175A-TPLE/TLP175A-TPLECT-ND/4562904" H 7600 2945 60  0001 C CNN "PurchasingLink"
+	1    7500 2450
+	1    0    0    -1
+$EndComp
+$Comp
+L D_Schottky_SOD123 D4
+U 1 1 59F8AACE
+P 6350 2950
+F 0 "D4" H 6350 3050 50  0000 C CNN
+F 1 "D_Schottky_SOD123" H 6350 2850 50  0000 C CNN
+F 2 "footprints:D_SOD-123W_OEM" H 6250 2950 50  0001 C CNN
+F 3 "https://assets.nexperia.com/documents/data-sheet/PMEG10010ELR.pdf" H 6350 3050 50  0001 C CNN
+F 4 "1727-2394-1-ND" H 6450 3150 60  0001 C CNN "MPN"
+F 5 "Digi-Key" H 6550 3250 60  0001 C CNN "MFN"
+F 6 "https://www.digikey.com/product-detail/en/nexperia-usa-inc/PMEG10010ELRX/1727-2394-1-ND/5436140" H 6650 3350 60  0001 C CNN "PurchasingLink"
+	1    6350 2950
+	-1   0    0    1
+$EndComp
+$Comp
+L D_Schottky_SOD123 D5
+U 1 1 59F8ADAC
+P 7200 3750
+F 0 "D5" H 7200 3850 50  0000 C CNN
+F 1 "D_Schottky_SOD123" H 7200 3650 50  0000 C CNN
+F 2 "footprints:D_SOD-123W_OEM" H 7100 3750 50  0001 C CNN
+F 3 "https://assets.nexperia.com/documents/data-sheet/PMEG10010ELR.pdf" H 7200 3850 50  0001 C CNN
+F 4 "1727-2394-1-ND" H 7300 3950 60  0001 C CNN "MPN"
+F 5 "Digi-Key" H 7400 4050 60  0001 C CNN "MFN"
+F 6 "https://www.digikey.com/product-detail/en/nexperia-usa-inc/PMEG10010ELRX/1727-2394-1-ND/5436140" H 7500 4150 60  0001 C CNN "PurchasingLink"
+	1    7200 3750
+	-1   0    0    1
+$EndComp
+$Comp
+L D_Schottky_SOD123 D6
+U 1 1 59F8B440
+P 7400 4400
+F 0 "D6" H 7400 4500 50  0000 C CNN
+F 1 "D_Schottky_SOD123" H 7400 4300 50  0000 C CNN
+F 2 "footprints:D_SOD-123W_OEM" H 7300 4400 50  0001 C CNN
+F 3 "https://assets.nexperia.com/documents/data-sheet/PMEG10010ELR.pdf" H 7400 4500 50  0001 C CNN
+F 4 "1727-2394-1-ND" H 7500 4600 60  0001 C CNN "MPN"
+F 5 "Digi-Key" H 7600 4700 60  0001 C CNN "MFN"
+F 6 "https://www.digikey.com/product-detail/en/nexperia-usa-inc/PMEG10010ELRX/1727-2394-1-ND/5436140" H 7700 4800 60  0001 C CNN "PurchasingLink"
+	1    7400 4400
+	0    1    1    0
+$EndComp
 $EndSCHEMATC

Commit message: Tracing ready Layout
Connections:
- net at D6.1 (K), K1.5, U2.4: now also D5.2 (A); no longer D5.1 (K)
- net at D4.1 (K), Q1.1 (G), R4.1: now also D5.1 (K); no longer D5.2 (A)
Changed lines of the file:
@@
 F 6 "https://www.digikey.com/product-detail/en/nexperia-usa-inc/PMEG10010ELRX/1727-2394-1-ND/5436140" H 7500 4150 60  0001 C CNN "PurchasingLink"
 	1    7200 3750
-	-1   0    0    1
+	1    0    0    -1
 $EndComp
 $Comp

Commit message: preparing for v2
Parts:
- removed D4, D5: D_Schottky_SOD123, footprints:D_SOD-123W_OEM, symbol D_Schottky_SOD123
Connections:
- net at Q1.1 (G), R4.1: now also C1.1, R1.2
Other:
- moved on the sheet: C2, C3, C4, D1, D2, D3, F1, L1, R10, R2, R5, R6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
