File: templates/oem-kicad-template/oem-kicad-template.kicad_pcb (KiCad board)
At the start: 2 copper layers, 0 parts

Commit message: Progress
Other:
- net class Default: trace_width 0.1524 -> 0.254; via_dia 0.6 -> 0.6096; via_drill 0.4 -> 0.3048
- rule trace_min: 0.1524 -> 0.254
- rule via_min_drill: 0.3 -> 0.3048
- rule via_min_size: 0.4 -> 0.6096
Changed lines of the file:
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@@
   )
   (setup
-    (last_trace_width 0.1524)
+    (last_trace_width 0.254)
     (user_trace_width 0.254)
     (user_trace_width 0.508)
@@
     (zone_clearance 0.508)
     (zone_45_only no)
-    (trace_min 0.1524)
+    (trace_min 0.254)
     (segment_width 0.2)
     (edge_width 0.15)
-    (via_size 0.6)
-    (via_drill 0.4)
-    (via_min_size 0.4)
-    (via_min_drill 0.3)
+    (via_size 0.6096)
+    (via_drill 0.3048)
+    (via_min_size 0.6096)
+    (via_min_drill 0.3048)
     (uvia_size 0.3)
     (uvia_drill 0.1)
@@
   (net_class Default "This is the default net class."
     (clearance 0.1524)
-    (trace_width 0.1524)
-    (via_dia 0.6)
-    (via_drill 0.4)
+    (trace_width 0.254)
+    (via_dia 0.6096)
+    (via_drill 0.3048)
     (uvia_dia 0.3)
     (uvia_drill 0.1)
