File: boards/dashboard/FunctionalBoard/dashboard.sch (KiCad schematic (older format))
At the start: 43 parts, among them IC1 ATMEGA16M1, J1 micromatch_male_10, J2 micromatch_male_14, J3 micromatch_female_RA_6, P1 CONN_02X03, U1 CAN_Transceiver, U2 TPS561201, U3 LM3480, U4 CP2120, Y1 Crystal_SMD

Commit message: Progress
Connections:
- net CANH: now also J2.9; no longer J2.8
- net CANL: now also J2.8; no longer J2.9
- net SCL: no longer J2.14
- net SDA: no longer J2.13
- net START: no longer J2.12
Changed lines of the file:
@@
 Text GLabel 4650 6300 0    55   Input ~ 0
 START
-Text GLabel 5750 5450 0    55   Input ~ 0
-SCL
-Text GLabel 5750 5550 0    55   Input ~ 0
-SDA
 Text GLabel 5750 5750 0    55   Input ~ 0
 LED2
 Text GLabel 5750 5850 0    55   Input ~ 0
 LED1
+Text GLabel 5750 6050 0    55   Input ~ 0
+CANL
 Text GLabel 5750 5950 0    55   Input ~ 0
-CANL
-Text GLabel 5750 6050 0    55   Input ~ 0
 CANH
 Text GLabel 5750 6150 0    55   Input ~ 0
@@
 $EndComp
 NoConn ~ 3400 2850
-Text GLabel 5750 5650 0    55   Input ~ 0
-START
 Text GLabel 3400 3550 2    60   Input ~ 0
 CS

Commit message: Boards updated
Parts:
- J3: symbol micromatch_female_RA_6 -> micromatch_female_RA_6-RESCUE-dashboard
Changed lines of the file:
@@
 EESchema Schematic File Version 2
+LIBS:dashboard-rescue
 LIBS:power
 LIBS:device
@@
 	5660 6750 5750 6750
 $Comp
-L micromatch_female_RA_6 J3
+L micromatch_female_RA_6-RESCUE-dashboard J3
 U 1 1 5A2F3264
 P 5160 1220
