File: boards/BSPD/BSPD.sch (KiCad schematic (older format))
At the start: 40 parts, among them J1 micromatch_female_RA_6, J2 Ultrafit_2, K1 G5Q-1A4-DC5-5V, Q1 MMBF170, Q2 MMBF170, U1 TPS561201, U2 SN74LVC1G08, U3 MCP6001, U4 SN74LVC1G02, U5 SN74LVC1G02

Commit message: BSPD Schematic and Layout Finalized to be checked off
Parts:
- removed J1: micromatch_female_RA_6, footprints:micromatch_female_ra_6, symbol micromatch_female_RA_6
- removed J2: Ultrafit_2, footprints:Ultrafit_2, symbol Ultrafit_2
- removed Q1, Q2: MMBF170, TO_SOT_Packages_SMD:SOT-23, symbol MMBF170
- added D1: D_Zener_18V, footprints:DO-214AA, symbol D_Zener_18V
- added J1: micromatch_female_RA_20, footprints:micromatch_female_ra_20, symbol micromatch_female_RA_20
- added Q1, Q2: SSM3K333R, footprints:SOT-23F, symbol SSM3K333R
- renumbered D1 to D2, D2 to D3, D3 to D4, D4 to D5, D5 to D6
Connections:
- net +12V: now also D1.1 (K), J1.2
- net 12V_Fused: now also U1.3 (VIN)
- net GND: now also D1.2 (A), J1.1, Q1.2 (S)
- net VCC: now also J1.5
- net at R2.2, U1.5 (EN): no longer U1.3 (VIN)
- net ShutdownOut: now reaches K1.2
- net ShutdownOut: now also J1.13, J1.14, J1.15, J1.16, J1.17, J1.18
- net ShutdownIn: now reaches K1.3
- net ShutdownIn: now also J1.10, J1.11, J1.12, J1.7, J1.8, J1.9
- net at D6.2 (A), K1.1: now also Q2.3 (D)
- net at R4.2, U2.1 (in): now also J1.4, J1.6
- net at R3.1, U2.2 (in): now also J1.3
- net BSPDRelaySense: now reaches R16.1, U4.1 (in), U5.4 (out)
- net BSPDRelaySense: now also J1.19, Q2.1 (G)
- net at R8.1, U4.2 (in): now also Q1.3 (D)
- net at C3.1, R6.2: now also Q1.1 (G)
- net at R17.1: now also Q2.2 (S)
- no-connect marks 0 -> 1

Commit message: Checked off BSPD Schematic and Layout
Parts:
- C1: footprint Capacitors_SMD:C_1206 -> footprints:C_1206_OEM
- C2, C4: footprint Capacitors_SMD:C_0805 -> footprints:C_0805_OEM
- D2, D4: footprint LEDs:LED_0805 -> footprints:LED_0805_OEM
- R1, R11, R2, R5, R7: footprint Resistors_SMD:R_0805 -> footprints:R_0805_OEM
- R9: footprint Resistors_SMD:R_2512 -> footprints:R_2512_OEM
- U1: footprint TO_SOT_Packages_SMD:SOT-23-6 -> footprints:SOT-23-6_OEM
- U3: footprint TO_SOT_Packages_SMD:SOT-23-5 -> footprints:SOT-23-5_OEM
Connections:
- net BSPDRelaySense: now also R17.1
- net GND: now also Q2.2 (S)
Other:
- moved on the sheet: R17
Changed lines of the file:
@@
 F 0 "R2" V 1680 1400 50  0000 C CNN
 F 1 "R_10k" V 1500 1400 50  0000 C CNN
-F 2 "Resistors_SMD:R_0805" H 1530 1400 50  0001 C CNN
+F 2 "footprints:R_0805_OEM" H 1530 1400 50  0001 C CNN
 F 3 "http://www.bourns.com/data/global/pdfs/CRS.pdf" H 1680 1400 50  0001 C CNN
 F 4 "CRS0805-FX-1002ELFCT-ND" H 1600 1400 60  0001 C CNN "MPN"
@@
 F 0 "R5" V 2730 1550 50  0000 C CNN
 F 1 "R_10k" V 2550 1550 50  0000 C CNN
-F 2 "Resistors_SMD:R_0805" H 2580 1550 50  0001 C CNN
+F 2 "footprints:R_0805_OEM" H 2580 1550 50  0001 C CNN
 F 3 "http://www.bourns.com/data/global/pdfs/CRS.pdf" H 2730 1550 50  0001 C CNN
 F 4 "CRS0805-FX-1002ELFCT-ND" H 2650 1550 60  0001 C CNN "MPN"
@@
 F 0 "R1" V 1180 1550 50  0000 C CNN
 F 1 "R_1k" V 1000 1550 50  0000 C CNN
-F 2 "Resistors_SMD:R_0805" H 1030 1550 50  0001 C CNN
+F 2 "footprints:R_0805_OEM" H 1030 1550 50  0001 C CNN
 F 3 "https://www.seielect.com/Catalog/SEI-rncp.pdf" H 1180 1550 50  0001 C CNN
 F 4 "Digi-Key" H 1100 1550 60  0001 C CNN "MFN"
@@
 F 0 "R7" V 2750 1400 50  0000 C CNN
 F 1 "R_55.1k" V 2950 1400 50  0000 C CNN
-F 2 "Resistors_SMD:R_0805" H 2780 1400 50  0001 C CNN
+F 2 "footprints:R_0805_OEM" H 2780 1400 50  0001 C CNN
 F 3 "http://www.yageo.com.tw/exep/pages/download/literatures/PYu-R_INT-thick_7.pdf" H 2930 1400 50  0001 C CNN
 F 4 "311-51.1KCRCT-ND" H 2850 1400 60  0001 C CNN "MPN"
@@
 F 0 "R11" V 3800 1350 50  0000 C CNN
 F 1 "R_200" V 4000 1350 50  0000 C CNN
-F 2 "Resistors_SMD:R_0805" H 3830 1350 50  0001 C CNN
+F 2 "footprints:R_0805_OEM" H 3830 1350 50  0001 C CNN
 F 3 "https://www.seielect.com/Catalog/SEI-RMCF_RMCP.pdf" H 3980 1350 50  0001 C CNN
 F 4 "Digi-Key" H 3900 1350 60  0001 C CNN "MFN"
@@
 F 0 "R9" V 3630 1200 50  0000 C CNN
 F 1 "R_0_Jumper" V 3450 1200 50  0000 C CNN
-F 2 "Resistors_SMD:R_2512" H 3480 1200 50  0001 C CNN
+F 2 "footprints:R_2512_OEM" H 3480 1200 50  0001 C CNN
 F 3 "http://www.te.com/commerce/DocumentDelivery/DDEController?Action=srchrtrv&DocNm=9-1773463-7&DocType=DS&DocLang=English" H 3630 1200 50  0001 C CNN
 F 4 "A121322CT-ND" H 3550 1200 60  0001 C CNN "MPN"
@@
 F 0 "D2" H 1100 1750 50  0000 C CNN
 F 1 "LED_0805" H 1100 1950 50  0000 C CNN
-F 2 "LEDs:LED_0805" H 1000 1850 50  0001 C CNN
+F 2 "footprints:LED_0805_OEM" H 1000 1850 50  0001 C CNN
 F 3 "http://www.osram-os.com/Graphics/XPic9/00078860_0.pdf" H 1100 1950 50  0001 C CNN
 F 4 "475-1410-1-ND" H 1100 1850 60  0001 C CNN "MPN"
@@
 F 0 "D4" H 3900 1550 50  0000 C CNN
 F 1 "LED_0805" H 3900 1750 50  0000 C CNN
-F 2 "LEDs:LED_0805" H 3800 1650 50  0001 C CNN
+F 2 "footprints:LED_0805_OEM" H 3800 1650 50  0001 C CNN
 F 3 "http://www.osram-os.com/Graphics/XPic9/00078860_0.pdf" H 3900 1750 50  0001 C CNN
 F 4 "475-1410-1-ND" H 3900 1650 60  0001 C CNN "MPN"
@@
 F 0 "C2" H 2850 950 50  0000 L CNN
 F 1 "C_0.1uF" H 2850 1150 50  0000 L CNN
-F 2 "Capacitors_SMD:C_0805" H 2838 900 50  0001 C CNN
+F 2 "footprints:C_0805_OEM" H 2838 900 50  0001 C CNN
 F 3 "http://datasheets.avx.com/X7RDielectric.pdf" H 2825 1150 50  0001 C CNN
 F 4 "478-3352-1-ND" H 2800 1050 60  0001 C CNN "MPN"
@@
 F 0 "C1" H 1375 1650 50  0000 L CNN
 F 1 "C_22uF" H 1375 1450 50  0000 L CNN
-F 2 "Capacitors_SMD:C_1206" H 1388 1400 50  0001 C CNN
+F 2 "footprints:C_1206_OEM" H 1388 1400 50  0001 C CNN
 F 3 "http://www.samsungsem.com/kr/support/product-search/mlcc/__icsFiles/afieldfile/2017/07/28/S_CL31A226KOCLFNC.pdf" H 1375 1650 50  0001 C CNN
 F 4 "1276-2725-1-ND" H 1350 1550 60  0001 C CNN "MPN"
@@
 F 0 "C4" H 3425 1650 50  0000 L CNN
 F 1 "C_47uF" H 3425 1450 50  0000 L CNN
-F 2 "Capacitors_SMD:C_0805" H 3438 1400 50  0001 C CNN
+F 2 "footprints:C_0805_OEM" H 3438 1400 50  0001 C CNN
 F 3 "http://www.yuden.co.jp/productdata/catalog/en/mlcc_all_e.pdf" H 3425 1650 50  0001 C CNN
 F 4 "587-4280-1-ND" H 3400 1550 60  0001 C CNN "MPN"
@@
 F 0 "U3" H 5250 3600 50  0000 C CNN
 F 1 "MCP6001" H 5400 3200 50  0000 C CNN
-F 2 "TO_SOT_Packages_SMD:SOT-23-5" H 5150 3500 50  0001 C CNN
+F 2 "footprints:SOT-23-5_OEM" H 5150 3500 50  0001 C CNN
 F 3 "" H 5250 3600 50  0000 C CNN
 	1    5200 3400
@@
 L R_10k R17
 U 1 1 5A0B863B
-P 7885 3915
-F 0 "R17" V 7965 3915 50  0000 C CNN
-F 1 "R_10k" V 7785 3915 50  0000 C CNN
-F 2 "footprints:R_0805_OEM" H 7815 3915 50  0001 C CNN
-F 3 "http://www.bourns.com/data/global/pdfs/CRS.pdf" H 7965 3915 50  0001 C CNN
-F 4 "CRS0805-FX-1002ELFCT-ND" H 7885 3915 60  0001 C CNN "MPN"
-F 5 "Digi-Key" H 7885 3915 60  0001 C CNN "MFN"
-F 6 "Value" H 7885 3915 60  0001 C CNN "Package"
-F 7 "https://www.digikey.com/products/en?keywords=CRS0805-FX-1002ELFCT-ND" H 8365 4315 60  0001 C CNN "PurchasingLink"
-	1    7885 3915
-	1    0    0    -1
-$EndComp
-Wire Wire Line
-	7885 4065 7885 4205
+P 7555 3800
+F 0 "R17" V 7635 3800 50  0000 C CNN
+F 1 "R_10k" V 7455 3800 50  0000 C CNN
+F 2 "footprints:R_0805_OEM" H 7485 3800 50  0001 C CNN
+F 3 "http://www.bourns.com/data/global/pdfs/CRS.pdf" H 7635 3800 50  0001 C CNN
+F 4 "CRS0805-FX-1002ELFCT-ND" H 7555 3800 60  0001 C CNN "MPN"
+F 5 "Digi-Key" H 7555 3800 60  0001 C CNN "MFN"
+F 6 "Value" H 7555 3800 60  0001 C CNN "Package"
+F 7 "https://www.digikey.com/products/en?keywords=CRS0805-FX-1002ELFCT-ND" H 8035 4200 60  0001 C CNN "PurchasingLink"
+	1    7555 3800
+	1    0    0    -1
+$EndComp
+Wire Wire Line
+	7885 3660 7885 3800
 $Comp
 L GND #PWR031
 U 1 1 5A0B8864
-P 7885 4205
-F 0 "#PWR031" H 7885 3955 50  0001 C CNN
-F 1 "GND" H 7885 4055 50  0000 C CNN
-F 2 "" H 7885 4205 50  0000 C CNN
-F 3 "" H 7885 4205 50  0000 C CNN
-	1    7885 4205
+P 7885 3800
+F 0 "#PWR031" H 7885 3550 50  0001 C CNN
+F 1 "GND" H 7885 3650 50  0000 C CNN
+F 2 "" H 7885 3800 50  0000 C CNN
+F 3 "" H 7885 3800 50  0000 C CNN
+	1    7885 3800
 	1    0    0    -1
 $EndComp
@@
 Text Label 1735 4850 0    60   ~ 0
 BSPDRelaySense
-Text Label 7505 4715 0    60   ~ 0
+Text Label 7375 5505 0    60   ~ 0
 BSPDRelaySense
 $Comp
@@
 Wire Wire Line
 	6955 3460 7585 3460
-Connection ~ 7505 3460
-Wire Wire Line
-	7505 3460 7505 4715
-Wire Wire Line
-	7885 3765 7885 3660
 Wire Wire Line
 	7885 2130 7885 3260
@@
 F 0 "U1" H 2000 1000 60  0000 C CNN
 F 1 "TPS561201" H 2200 1650 60  0000 C CNN
-F 2 "TO_SOT_Packages_SMD:SOT-23-6" H 1900 1550 60  0001 C CNN
+F 2 "footprints:SOT-23-6_OEM" H 1900 1550 60  0001 C CNN
 F 3 "http://www.ti.com/lit/ds/symlink/tps561201.pdf" H 2000 1650 60  0001 C CNN
 F 4 "Digi-Key" H 2200 1300 60  0001 C CNN "MFN"
@@
 	1    0    0    -1
 $EndComp
+Connection ~ 7555 3460
+Wire Wire Line
+	7555 3460 7555 3650
+Wire Wire Line
+	7555 3950 7555 4065
+$Comp
+L GND #PWR039
+U 1 1 5A2F55FF
+P 7555 4065
+F 0 "#PWR039" H 7555 3815 50  0001 C CNN
+F 1 "GND" H 7555 3915 50  0000 C CNN
+F 2 "" H 7555 4065 50  0000 C CNN
+F 3 "" H 7555 4065 50  0000 C CNN
+	1    7555 4065
+	1    0    0    -1
+$EndComp
+Wire Wire Line
+	7375 3460 7375 5505
+Connection ~ 7375 3460
 $EndSCHEMATC

Commit message: Labeling for ESF
Parts:
- removed C5: C_1uF, footprints:C_0805_OEM, symbol C_1uF
- added C5: C_10uF, footprints:C_0805_OEM, symbol C_10uF
Connections:
- net GND: now also C5.2
- net at R12.1, U3.3 (+): now also C5.1
Other:
- note added: "Brake Sensor Input\n\n"
- note added: "Current Sensor Input"
- note added: "OP-AMP Timer"
- note added: "RS-NOR Latch"
Changed lines of the file:
@@
 Wire Wire Line
 	1600 3550 1750 3550
-Wire Wire Line
-	1750 3550 1750 3500
 $Comp
 L VCC #PWR016
 U 1 1 5A0B3095
-P 1750 3500
-F 0 "#PWR016" H 1750 3350 50  0001 C CNN
-F 1 "VCC" H 1750 3650 50  0000 C CNN
-F 2 "" H 1750 3500 50  0000 C CNN
-F 3 "" H 1750 3500 50  0000 C CNN
-	1    1750 3500
+P 1750 3550
+F 0 "#PWR016" H 1750 3400 50  0001 C CNN
+F 1 "VCC" H 1750 3700 50  0000 C CNN
+F 2 "" H 1750 3550 50  0000 C CNN
+F 3 "" H 1750 3550 50  0000 C CNN
+	1    1750 3550
 	1    0    0    -1
 $EndComp
@@
 P 6625 3460
 F 0 "U5" H 7025 3810 60  0000 C CNN
-F 1 "SN74LVC1G02" H 7025 3910 60  0000 C CNN
+F 1 "SN74LVC1G02" H 6205 3665 60  0000 C CNN
 F 2 "footprints:SOT-23-5_OEM" H 6625 3460 60  0001 C CNN
 F 3 "" H 6625 3460 60  0000 C CNN
@@
 P 6320 4720
 F 0 "U4" H 6720 5070 60  0000 C CNN
-F 1 "SN74LVC1G02" H 6720 5170 60  0000 C CNN
+F 1 "SN74LVC1G02" H 6580 4910 60  0000 C CNN
 F 2 "footprints:SOT-23-5_OEM" H 6320 4720 60  0001 C CNN
 F 3 "" H 6320 4720 60  0000 C CNN
@@
 Connection ~ 6870 2130
 $Comp
-L C_1uF C5
-U 1 1 5A1B7D2C
-P 4450 3700
-F 0 "C5" H 4475 3800 50  0000 L CNN
-F 1 "C_1uF" H 4475 3600 50  0000 L CNN
-F 2 "footprints:C_0805_OEM" H 4488 3550 50  0001 C CNN
-F 3 "http://datasheets.avx.com/X7RDielectric.pdf" H 4475 3800 50  0001 C CNN
-F 4 "CAP CER 1UF 25V X7R 0805" H 4975 4300 60  0001 C CNN "Description"
-F 5 "478-10487-1-ND" H 4450 3700 60  0001 C CNN "MPN"
-F 6 "Digi-Key" H 4450 3700 60  0001 C CNN "MFN"
-F 7 "Value" H 4450 3700 60  0001 C CNN "Package"
-F 8 "https://www.digikey.com/product-detail/en/avx-corporation/08053C105JAT2A/478-10487-1-ND/6797628" H 4875 4200 60  0001 C CNN "PurchasingLink"
-	1    4450 3700
-	1    0    0    -1
-$EndComp
-$Comp
 L R_71.5k R12
 U 1 1 5A1B8CFF
@@
 	7375 3460 7375 5505
 Connection ~ 7375 3460
+Text Notes 1755 2720 0    60   ~ 0
+Brake Sensor Input\n\n
+Text Notes 1410 3350 0    60   ~ 0
+Current Sensor Input
+$Comp
+L C_10uF C5
+U 1 1 5A4E9EC4
+P 4450 3700
+F 0 "C5" H 4475 3800 50  0000 L CNN
+F 1 "C_10uF" H 4475 3600 50  0000 L CNN
+F 2 "footprints:C_0805_OEM" H 4488 3550 50  0001 C CNN
+F 3 "http://datasheets.avx.com/cx5r.pdf" H 4475 3800 50  0001 C CNN
+F 4 "478-5167-1-ND" H 4450 3700 60  0001 C CNN "MPN"
+F 5 "Digi-Key" H 4450 3700 60  0001 C CNN "MFN"
+F 6 "Value" H 4450 3700 60  0001 C CNN "Package"
+F 7 "https://www.digikey.com/product-detail/en/avx-corporation/0805ZD106KAT2A/478-5167-1-ND/1913257" H 4875 4200 60  0001 C CNN "PurchasingLink"
+	1    4450 3700
+	1    0    0    -1
+$EndComp
+Text Notes 4430 2665 0    60   ~ 0
+OP-AMP Timer
+Wire Notes Line
+	3835 2710 5510 2710
+Wire Notes Line
+	5510 2710 5510 4495
+Wire Notes Line
+	5510 4495 3830 4495
+Wire Notes Line
+	3830 4495 3830 2710
+Text Notes 5980 2850 0    60   ~ 0
+RS-NOR Latch
+Wire Notes Line
+	6940 2930 6940 5290
+Wire Notes Line
+	6940 5290 6065 5290
+Wire Notes Line
+	6065 5290 6065 2930
+Wire Notes Line
+	6065 2930 6940 2930
+Wire Notes Line
+	6940 2935 6935 2935
 $EndSCHEMATC

Commit message: Updated info for BOM
Parts:
- R12: MFN (none) -> Yageo; MPN (none) -> RC0805FR-0771K5L; Package (none) -> Value; PurchasingLink (none) -> https://www.digikey.com/product-detail/en/yageo/RC0805FR-07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
- U2: MFN (none) -> Texas Instruments; MPN (none) -> SN74LVC1G08DBVR; Package (none) -> SC-74A, SOT-753; PurchasingLink (none) -> https://www.digikey.com/product-detail/en/texas-instruments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
- U3: MNF (none) -> Microchip Technology; MPN (none) -> MCP6001T-I/OT; Package (none) -> SC-74A, SOT-753; PurchasingLink (none) -> https://www.digikey.com/product-detail/en/microchip-technol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
- U4, U5: MFN (none) -> Texas Instruments; MPN (none) -> SN74LVC1G02DBVR; Package (none) -> SC-74A, SOT-753; PurchasingLink (none) -> https://www.digikey.com/product-detail/en/texas-instruments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
Changed lines of the file:
@@
 F 1 "SN74LVC1G08" H 3700 3550 60  0000 C CNN
 F 2 "footprints:SOT-23-5_OEM" H 3350 3300 60  0001 C CNN
-F 3 "" H 3350 3300 60  0000 C CNN
+F 3 "http://www.ti.com/lit/ds/symlink/sn74lvc1g08.pdf" H 4930 4380 60  0001 C CNN
+F 4 "SN74LVC1G08DBVR " H 3250 3300 60  0001 C CNN "MPN"
+F 5 "Texas Instruments" H 3250 3300 60  0001 C CNN "MFN"
+F 6 "SC-74A, SOT-753" H 3250 3300 60  0001 C CNN "Package"
+F 7 "https://www.digikey.com/product-detail/en/texas-instruments/SN74LVC1G08DBVR/296-11601-1-ND/385740" H 3250 3300 60  0001 C CNN "PurchasingLink"
 	1    3250 3300
 	1    0    0    -1
@@
 F 1 "MCP6001" H 5400 3200 50  0000 C CNN
 F 2 "footprints:SOT-23-5_OEM" H 5150 3500 50  0001 C CNN
-F 3 "" H 5250 3600 50  0000 C CNN
+F 3 "http://ww1.microchip.com/downloads/en/DeviceDoc/21733j.pdf" H 5250 3600 50  0000 C CNN
+F 4 " MCP6001T-I/OT" H 5200 3400 60  0001 C CNN "MPN"
+F 5 "Microchip Technology" H 5200 3400 60  0001 C CNN "MNF"
+F 6 "SC-74A, SOT-753 " H 5200 3400 60  0001 C CNN "Package"
+F 7 "https://www.digikey.com/product-detail/en/microchip-technology/MCP6001T-I-OT/MCP6001T-I-OTCT-ND/697158" H 5200 3400 60  0001 C CNN "PurchasingLink"
 	1    5200 3400
 	1    0    0    -1
@@
 F 1 "SN74LVC1G02" H 6205 3665 60  0000 C CNN
 F 2 "footprints:SOT-23-5_OEM" H 6625 3460 60  0001 C CNN
-F 3 "" H 6625 3460 60  0000 C CNN
+F 3 "http://www.ti.com/lit/ds/symlink/sn74lvc1g02.pdf" H 6625 3460 60  0001 C CNN
+F 4 "SN74LVC1G02DBVR" H 6625 3460 60  0001 C CNN "MPN"
+F 5 "Texas Instruments" H 6625 3460 60  0001 C CNN "MFN"
+F 6 "SC-74A, SOT-753" H 6625 3460 60  0001 C CNN "Package"
+F 7 "https://www.digikey.com/product-detail/en/texas-instruments/SN74LVC1G02DBVR/296-11597-1-ND/385736" H 6625 3460 60  0001 C CNN "PurchasingLink"
 	1    6625 3460
 	1    0    0    -1
@@
 F 1 "SN74LVC1G02" H 6580 4910 60  0000 C CNN
 F 2 "footprints:SOT-23-5_OEM" H 6320 4720 60  0001 C CNN
-F 3 "" H 6320 4720 60  0000 C CNN
+F 3 "http://www.ti.com/lit/ds/symlink/sn74lvc1g02.pdf" H 6320 4720 60  0000 C CNN
+F 4 "SN74LVC1G02DBVR" H 6320 4720 60  0001 C CNN "MPN"
+F 5 "Texas Instruments" H 6320 4720 60  0001 C CNN "MFN"
+F 6 " SC-74A, SOT-753 " H 6320 4720 60  0001 C CNN "Package"
+F 7 "https://www.digikey.com/product-detail/en/texas-instruments/SN74LVC1G02DBVR/296-11597-1-ND/385736" H 6320 4720 60  0001 C CNN "PurchasingLink"
 	1    6320 4720
 	1    0    0    -1
@@
 	5890 4660 5890 4135
 Wire Wire Line
-	5890 4135 7030 4135
-Wire Wire Line
-	7030 4135 7030 3455
+	7030 4135 5890 4135
+Wire Wire Line
+	7030 3455 7030 4135
 Wire Wire Line
 	3630 3300 3630 3475
@@
 $EndComp
 Wire Wire Line
-	7885 2130 7580 2130
+	7580 2130 7885 2130
 $Comp
 L R_200 R10
@@
 $EndComp
 Wire Wire Line
-	6980 2130 6590 2130
+	6590 2130 6980 2130
 Wire Wire Line
 	6590 2130 6590 2025
@@
 F 1 "R_71.5k" V 3950 3300 50  0000 C CNN
 F 2 "footprints:R_0805_OEM" V 3980 3300 50  0001 C CNN
-F 3 "" H 4050 3300 50  0001 C CNN
+F 3 "http://www.yageo.com/documents/recent/PYu-RC_Group_51_RoHS_L_8.pdf" H 4050 3300 50  0001 C CNN
+F 4 "RC0805FR-0771K5L " V 4050 3300 60  0001 C CNN "MPN"
+F 5 "Yageo" V 4050 3300 60  0001 C CNN "MFN"
+F 6 "Value" V 4050 3300 60  0001 C CNN "Package"
+F 7 "https://www.digikey.com/product-detail/en/yageo/RC0805FR-0771K5L/311-71.5KCRCT-ND/731072" V 4050 3300 60  0001 C CNN "PurchasingLink"
 	1    4050 3300
 	0    1    1    0
@@
 $EndComp
 Wire Wire Line
-	3710 5390 2770 5390
+	2770 5390 3710 5390
 Wire Wire Line
 	2770 5390 2770 5250
