File: boards/Brake_Light_Shutdown_Sensing/Brake_Light_Shutdown_Sensing.kicad_pcb (KiCad board)
At the start: 2 copper layers, 84 parts, among them IC1 ATMEGA16M1, J1 micromatch_female_RA_6, J2 micromatch_female_RA_20, P1 CONN_02X03, P2 CONN_02X03, Q1 SSM3K333R, Q2 SSM3K333R, Q3 SSM3K333R, Q4 SSM3K333R, Q5 SSM3K333R, Q6 SSM3K333R, Q7 SSM3K333R, U1 MCP6001RT, U2 TPS561201, U3 ATMEGA328P-AU, U5 CAN_Transceiver, Y1 Crystal_SMD, Y2 Crystal_SMD

Commit message: Draft of Layout
Parts:
- moved D13 93.2 mm to (176.5, 104.4), turned to 90 degrees
- moved R32 90.4 mm to (174.4, 104.4), turned to 90 degrees
- moved D14 83.9 mm to (172.4, 104.4), turned to 90 degrees
- moved R33 80.8 mm to (170.4, 104.4), turned to 90 degrees
- moved D9 79.0 mm to (179.8, 133.4)
- moved Q7 79.0 mm to (173.4, 133.4)
- moved R27 79.0 mm to (178.5, 137.2)
- moved R29 79.0 mm to (177.2, 133.4)
- moved R31 79.0 mm to (173.4, 137.2)
- moved C3 78.7 mm to (160.7, 92.3)
- moved C6 78.7 mm to (166.8, 85.1)
- moved D1 78.7 mm to (152.1, 92.3)
- moved F1 78.7 mm to (156.7, 89.7)
- moved R11 78.7 mm to (175.0, 95.3)
- moved U2 78.7 mm to (166.8, 89.0)
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Routing:
- net VCC: track 2.84 -> 9.51 mm

Commit message: Updated Layout
Parts:
- added C13: C_1uF, footprints:C_0805_OEM, F.Cu at (177.7, 91.7)
- added C14: C_0.1uF, footprints:C_0805_OEM, F.Cu at (177.7, 93.8)
- moved U5 47.9 mm to (156.7, 126.3), turned to 180 degrees
- moved D5 45.0 mm to (204.4, 132.6)
- moved Q3 45.0 mm to (198.1, 132.6)
- moved R15 45.0 mm to (203.1, 136.4)
- moved R17 45.0 mm to (201.9, 132.6)
- moved R19 45.0 mm to (198.1, 136.4)
- moved C10 43.6 mm to (161.7, 126.5), turned to 270 degrees
- moved D6 34.0 mm to (175.7, 132.6)
- moved Q4 34.0 mm to (169.4, 132.6)
- moved R20 34.0 mm to (174.4, 136.4)
- moved R22 34.0 mm to (173.2, 132.6)
- moved R24 34.0 mm to (169.4, 136.4)
- moved D8 33.3 mm to (166.3, 132.6)
- moved Q6 33.3 mm to (160.0, 132.6)
- moved R26 33.3 mm to (165.0, 136.4)
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Connections:
- IC1 pad 13: /Brake_Light_Gate -> /R_EStop_Pin
- IC1 pad 14: /data2 -> /BSPD_Pin
- IC1 pad 15: /data1 -> /HVD_Pin
- IC1 pad 16: /HVD_Pin -> /TSMS_Pin
- IC1 pad 17: /L_E-Stop_Pin -> /LED_4
- IC1 pad 21: Net-(IC1-Pad21) -> (no net)
- IC1 pad 22: /LED_4 -> /data1
- IC1 pad 23: /BSPD_Out -> /data2
- IC1 pad 24: /data4 -> /data3
- IC1 pad 25: /Main_Shut_Fuse -> /data4
- IC1 pad 26: /TSMS_Pin -> /Brake_Light_Gate
- IC1 pad 27: /R_EStop_Pin -> /BSPD_Out
- IC1 pad 28: Net-(IC1-Pad28) -> /Analog_Brake_Sense
- IC1 pad 30: /BSPD_Pin -> Net-(IC1-Pad30)
- IC1 pad 32: /data3 -> (no net)
- IC1 pad 8: /Analog_Brake_Sense -> /Main_Shut_Fuse
- IC1 pad 9: /RESET -> /L_E-Stop_Pin
- J2 pad 10: /LED_1 -> /Brake_Light_LSD
- J2 pad 11: /LED_2 -> +5V
- J2 pad 12: /Brake_Light_LSD -> /Brake_Switch-
- J2 pad 13: +5V -> /BSPD_Out
- J2 pad 14: /Brake_Switch- -> /Analog_Brake_Sense
- J2 pad 15: /BSPD_Out -> /LED_1
- J2 pad 16: /BSPD_Stat_Out -> /LED_2
- J2 pad 17: /SDA -> /BSPD_Stat_Out
- J2 pad 18: /SCL -> /SDA
- J2 pad 19: /Analog_Brake_Sense -> /SCL
- J2 pad 20: Net-(J2-Pad20) -> (no net)
- P2 pad 1: /32 -> /MISO
- P2 pad 3: /SCK32 -> /SCK
- P2 pad 4: /MOSI32 -> /MOSI
- R38 pad 1: /LED_1 -> /LED_2
- R38 pad 2: Net-(IC1-Pad28) -> Net-(IC1-Pad30)
- R39 pad 1: /LED_2 -> /LED_1
- U3 pad 1: Net-(U3-Pad1) -> (no net)
- U3 pad 10: Net-(U3-Pad10) -> (no net)
- U3 pad 15: /MOSI32 -> /MOSI
- U3 pad 16: /MISO32 -> /MISO
- U3 pad 19: Net-(U3-Pad19) -> (no net)
- U3 pad 2: Net-(U3-Pad2) -> (no net)
- U3 pad 22: Net-(U3-Pad22) -> (no net)
- U3 pad 25: Net-(U3-Pad25) -> (no net)
- U3 pad 26: Net-(U3-Pad26) -> (no net)
- U3 pad 30: Net-(U3-Pad30) -> (no net)
- U3 pad 31: Net-(U3-Pad31) -> (no net)
- U3 pad 32: Net-(U3-Pad32) -> (no net)
- U3 pad 9: Net-(U3-Pad9) -> (no net)
- U5 pad 5: Net-(U5-Pad5) -> (no net)
Routing:
- net VCC: track 9.51 -> 2.84 mm
- net Net-(C13-Pad1): track 12.0 -> 17.6 mm
- net GND: track 56.5 -> 55.2 mm
Other:
- board outline added: 70 x 70 mm
- board text added: "Main"
