File: boards/wheel_speed_sensing/wheel_speed_sensing.sch (KiCad schematic (older format))
At the start: 34 parts

Commit message: A bit more work on the schematic
Parts:
- added J? (x4): Conn_01x03, symbol Conn_01x03
- added R? (x4): R_3k, footprints:R_0805_OEM, symbol R_3k
- added R? (x4): R_330, footprints:R_0805_OEM, symbol R_330
Connections:
- net GND: now also U?.11 (VCC-), R?.2, R?.2, R?.2, R?.2
- net SensorLeft1+: now also J?.2 (Pin_2); no longer IC?.16 ((PCINT2/ADC5/INT1/ACMPN0)PB2)
- net SensorLeft2+: now also J?.2 (Pin_2); no longer IC?.15 ((PCINT23/ACMP0)PD7)
- net SensorRight1+: now also J?.2 (Pin_2); no longer IC?.26 ((PCINT5/ADC6/INT2/ACMPN1/AMP2-)PB5)
- net SensorRight2+: now also J?.2 (Pin_2); no longer IC?.22 ((PCINT14/ADC10/ACMP1)PC6)
- net VCC: now also U?.4 (VCC+)
- net SensorLeft1+Final: now reaches U?.1 (Output1)
- net SensorLeft1+Final: now also IC?.16 ((PCINT2/ADC5/INT1/ACMPN0)PB2), J?.3 (Pin_3), R?.1
- net SensorRight1+Amp: now reaches U?.10 (Ch3+)
- net SensorRight1+Amp: now also J?.1 (Pin_1)
- net SensorRight2+Amp: now reaches U?.12 (Ch4+)
- net SensorRight2+Amp: now also J?.1 (Pin_1)
- net Ch4-: now reaches U?.13 (Ch4-)
- net Ch4-: now also R?.1, R?.2
- net SensorRight2+Final: now reaches U?.14 (Output4)
- net SensorRight2+Final: now also IC?.22 ((PCINT14/ADC10/ACMP1)PC6), J?.3 (Pin_3), R?.1
- net Ch1-: now reaches U?.2 (Ch1-)
- net Ch1-: now also R?.1, R?.2
- net SensorLeft1+Amp: now reaches U?.3 (Ch1+)
- net SensorLeft1+Amp: now also J?.1 (Pin_1)
- net SensorLeft2+Amp: now reaches U?.5 (Ch2+)
- net SensorLeft2+Amp: now also J?.1 (Pin_1)
- net Ch2-: now reaches U?.6 (Ch2-)
- net Ch2-: now also R?.1, R?.2
- net SensorLeft2+Final: now reaches U?.7 (Output2)
- net SensorLeft2+Final: now also IC?.15 ((PCINT23/ACMP0)PD7), J?.3 (Pin_3), R?.1
- net SensorRight1+Final: now reaches U?.8 (Output3)
- net SensorRight1+Final: now also IC?.26 ((PCINT5/ADC6/INT2/ACMPN1/AMP2-)PB5), J?.3 (Pin_3), R?.1
- net Ch3-: now reaches U?.9 (Ch3-)
- net Ch3-: now also R?.1, R?.2
Other:
- note removed: "Digital I/O pins say PCINT\nAnalog enabled pins say ADC"
- note removed: "It is best to add at least 2-3 programming\nLEDs on your board for troubleshooting.\nUse Net Labels (the hotkey is "L") to connect\npins on your schematic without using wires.\nStart by placing a connector and labelling all\nthe pins with net labels according to the\nboard interface sheet."
- note removed: "Make sure you add 2 200 ohm resistors\nfrom two separate I/O pins which go to\nLED 1 and 2 on your connector\nPlease refer to the Board Interface Sheet\nfor a full pinout of the connectors on your board"
- moved on the sheet: J?, R?, U?

Commit message: fixed schematic
Parts:
- added R? (x2): R_200, footprints:R_0805_OEM, symbol R_200
Connections:
- net Ch1-: now also R?.1, R?.2; no longer R?.1, R?.2
- net Ch2-: now also R?.1, R?.2; no longer R?.1, R?.2
- net Ch3-: now also R?.1, R?.2; no longer R?.1, R?.2
- net Ch4-: now also R?.1, R?.2; no longer R?.1, R?.2
- net GND: now also R?.2, R?.2, R?.2, R?.2; no longer R?.2, R?.2, R?.2, R?.2
- net LED1: now also R?.1; no longer IC?.8 ((PCINT0/MISO/PSCOUT2A)PB0)
- net LED2: now also R?.1; no longer IC?.9 ((PCINT1/MOSI/PSCOUT2B)PB1)
- net SensorLeft1+Final: now also R?.1; no longer R?.1
- net SensorLeft2+Final: now also R?.1; no longer R?.1
- net SensorRight1+Final: now also R?.1; no longer R?.1
- net SensorRight2+Final: now also R?.1; no longer R?.1
- new net: IC?.8 ((PCINT0/MISO/PSCOUT2A)PB0), R?.2
- new net: IC?.9 ((PCINT1/MOSI/PSCOUT2B)PB1), R?.2
Other:
- moved on the sheet: R?, U?

Commit message: schematic is maybe done
Parts:
- removed J? (x4): Conn_01x03, symbol Conn_01x03
- added C11, C8: C_0.1uF, footprints:C_0805_OEM, symbol C_0.1uF
- added C7: C_1uF, footprints:C_0805_OEM, symbol C_1uF
- J1: renamed from J?; footprint (none) -> Pin_Headers:Pin_Header_Straight_1x03_Pitch2.54mm
- gave numbers to parts that had none: 43
Connections:
- net CANhigh is gone; now on net CANH: J2.8
- net CANlow is gone; now on net CANL: J2.9
- net SensorLeft1+Amp is gone; now on net SensorLeft1+: U3.3 (Ch1+)
- net SensorLeft2+Amp is gone; now on net SensorLeft2+: U3.5 (Ch2+)
- net SensorRight1+Amp is gone; now on net SensorRight1+: U3.10 (Ch3+)
- net SensorRight2+Amp is gone; now on net SensorRight2+: U3.12 (Ch4+)
- net GND: now also C11.2, C7.2, C8.2
- net VCC: now also C11.1
- net at C6.1, L1.2, R8.2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: now also C7.1, C8.1
- no-connect marks 1 -> 14
Other:
- moved on the sheet: C6, J1, R3

Commit message: maybe finished part of layout, maybe not, dont know how to type stuff and put the edge in though
Connections:
- net ProgLED2: now also IC1.14 ((PCINT22/ADC3/INT0/ACMPN2)PD6); no longer IC1.24 ((PCINT4/AMP0+)PB4)
Changed lines of the file:
@@
 Text Label 5900 2950 0    60   ~ 0
 ProgLED1
-Text Label 5900 3050 0    60   ~ 0
-ProgLED2
 $Comp
 L Conn_01x03 J1
@@
 NoConn ~ 5900 4550
 NoConn ~ 5900 4950
-NoConn ~ 5900 5050
 NoConn ~ 1300 3100
 Wire Wire Line
@@
 	1    0    0    -1
 $EndComp
+NoConn ~ 5900 3050
+Text Label 6150 4900 0    60   ~ 0
+ProgLED2
+Wire Wire Line
+	5900 5050 6100 5050
+Wire Wire Line
+	6100 5050 6100 4900
+Wire Wire Line
+	6100 4900 6150 4900
 $EndSCHEMATC
