File: boards/dashboard/InternalInterface/InternalInterface.sch (KiCad schematic (older format))
At the start: 6 parts, among them J1 micromatch_female_RA_10, J2 Ultrafit_2, J3 Ultrafit_2, J4 Ultrafit_4, J5 Ultrafit_4, J6 Ultrafit_4

Commit message: Edited interface boards
Connections:
- net GND: now also J1.2; no longer J1.3
- net START: now also J1.3; no longer J1.2
- net AMD renamed AMS
- net AMS: now also J1.4; no longer J1.6
- net IMS renamed IMD
- net IMD: now also J1.6; no longer J1.4
Changed lines of the file:
@@
 	1    0    0    -1
 $EndComp
-Text GLabel 1500 1720 2    60   BiDi ~ 0
+Text GLabel 1500 1820 2    60   BiDi ~ 0
 START
 Text GLabel 1500 1920 2    60   BiDi ~ 0
-IMS
+AMS
 Text GLabel 1500 2120 2    60   BiDi ~ 0
-AMD
+IMD
 Text GLabel 1500 2420 2    60   BiDi ~ 0
 SDA
@@
 L GND #PWR07
 U 1 1 5A28DFF4
-P 1580 1820
-F 0 "#PWR07" H 1580 1570 50  0001 C CNN
-F 1 "GND" H 1580 1670 50  0000 C CNN
-F 2 "" H 1580 1820 50  0001 C CNN
-F 3 "" H 1580 1820 50  0001 C CNN
-	1    1580 1820
+P 1580 1720
+F 0 "#PWR07" H 1580 1470 50  0001 C CNN
+F 1 "GND" H 1580 1570 50  0000 C CNN
+F 2 "" H 1580 1720 50  0001 C CNN
+F 3 "" H 1580 1720 50  0001 C CNN
+	1    1580 1720
 	0    -1   -1   0
 $EndComp
@@
 	1580 1620 1500 1620
 Wire Wire Line
-	1580 1820 1500 1820
-Wire Wire Line
 	1580 2020 1500 2020
 Wire Wire Line
@@
 	1580 2320 1500 2320
 Text GLabel 2720 1850 0    60   BiDi ~ 0
-IMS
+IMD
 Text GLabel 2690 2460 0    60   BiDi ~ 0
-AMD
+AMS
 $Comp
 L GND #PWR010
@@
 	-1   0    0    1
 $EndComp
+Wire Wire Line
+	1500 1720 1580 1720
 $EndSCHEMATC

Commit message: Boards updated
Parts:
- removed J1: micromatch_female_RA_10, footprints:micromatch_female_ra_10, symbol micromatch_female_RA_10
- added J1: micromatch_female_TOP_ENTRY_locking_10, footprints:micromatch_female_vert_10, symbol micromatch_female_TOP_ENTRY_locking_10
- added R1: R_200, footprints:R_0805_OEM, symbol R_200
Connections:
- net +5V: now also J1.1, J1.8, R1.2; no longer J6.3
- net AMS: now also J1.4
- net GND: now also J1.2, J1.5, J1.7
- net IMD: now also J1.6
- net SCL: now also J1.10
- net SDA: now also J1.9
- net START: now also J1.3
- new net: J6.3, R1.1
Changed lines of the file:
@@
 Comment4 ""
 $EndDescr
-$Comp
-L micromatch_female_RA_10 J1
-U 1 1 5A28D92D
-P 1350 2720
-F 0 "J1" H 1250 3920 60  0000 C CNN
-F 1 "micromatch_female_RA_10" H 1300 2770 60  0000 C CNN
-F 2 "footprints:micromatch_female_ra_10" H 1150 3820 60  0001 C CNN
-F 3 "" H 1250 3920 60  0001 C CNN
-F 4 "https://www.digikey.com/product-detail/en/te-connectivity-amp-connectors/1-338070-0/A99485CT-ND/1955787" H 1350 4020 60  0001 C CNN "PurchasingLink"
-F 5 "Digi-Key" H 1450 4120 60  0001 C CNN "MFN"
-F 6 "A99485CT-ND" H 1550 4220 60  0001 C CNN "MPN"
-F 7 "Value" H 1650 4320 60  0001 C CNN "Package"
-	1    1350 2720
-	1    0    0    -1
-$EndComp
 Text GLabel 1500 1820 2    60   BiDi ~ 0
 START
@@
 L +5V #PWR017
 U 1 1 5A28E3A4
-P 3370 2660
-F 0 "#PWR017" H 3370 2510 50  0001 C CNN
-F 1 "+5V" H 3370 2800 50  0000 C CNN
-F 2 "" H 3370 2660 50  0001 C CNN
-F 3 "" H 3370 2660 50  0001 C CNN
-	1    3370 2660
+P 3070 2660
+F 0 "#PWR017" H 3070 2510 50  0001 C CNN
+F 1 "+5V" H 3070 2800 50  0000 C CNN
+F 2 "" H 3070 2660 50  0001 C CNN
+F 3 "" H 3070 2660 50  0001 C CNN
+	1    3070 2660
 	0    -1   -1   0
 $EndComp
@@
 Wire Wire Line
 	1500 1720 1580 1720
+$Comp
+L R_200 R1
+U 1 1 5A7E6031
+P 3220 2660
+F 0 "R1" V 3300 2660 50  0000 C CNN
+F 1 "R_200" V 3120 2660 50  0000 C CNN
+F 2 "footprints:R_0805_OEM" H 3150 2660 50  0001 C CNN
+F 3 "https://www.seielect.com/Catalog/SEI-RMCF_RMCP.pdf" H 3300 2660 50  0001 C CNN
+F 4 "Digi-Key" H 3220 2660 60  0001 C CNN "MFN"
+F 5 "RMCF0805JT200RCT-ND" H 3220 2660 60  0001 C CNN "MPN"
+F 6 "Value" H 3220 2660 60  0001 C CNN "Package"
+F 7 "https://www.digikey.com/products/en?keywords=RMCF0805JT200RCT-ND" H 3700 3060 60  0001 C CNN "PurchasingLink"
+	1    3220 2660
+	0    1    1    0
+$EndComp
+$Comp
+L micromatch_female_TOP_ENTRY_locking_10 J1
+U 1 1 5A80658E
+P 1350 2720
+F 0 "J1" H 1250 3920 60  0000 C CNN
+F 1 "micromatch_female_TOP_ENTRY_locking_10" H 1300 2770 60  0000 C CNN
+F 2 "footprints:micromatch_female_vert_10" H 1150 3820 60  0001 C CNN
+F 3 "http://www.te.com/commerce/DocumentDelivery/DDEController?Action=srchrtrv&DocNm=338068&DocType=Customer+Drawing&DocLang=English" H 1250 3920 60  0001 C CNN
+F 4 "https://www.digikey.com/product-detail/en/te-connectivity-amp-connectors/1-338068-0/A99504CT-ND/1955737" H 1350 4020 60  0001 C CNN "PurchasingLink"
+F 5 "Digi-Key" H 1450 4120 60  0001 C CNN "MFN"
+F 6 "A99504CT-ND" H 1550 4220 60  0001 C CNN "MPN"
+F 7 "Value" H 1650 4320 60  0001 C CNN "Package"
+	1    1350 2720
+	1    0    0    -1
+$EndComp
 $EndSCHEMATC
