File: boards/dashboard/dashboard_rev2/dashboard_rev2.kicad_pcb (KiCad board)
At the start: 2 copper layers, 87.9 x 50.6 mm, 51 parts, among them IC1 ATMEGA16M1, J1 micromatch_male_10, J2 micromatch_male_14, J3 micromatch_female_RA_6, J4 NanoFit_2, P1 CONN_02X03, P2 CONN_02X03, U1 CAN_Transceiver, U2 TPS561201, U3 ATMEGA328P-AU, Y1 Crystal_SMD, Y2 Crystal_SMD

Commit message: Gerbers and PDFs
Connections:
- C10 pad 2: Net-(C10-Pad2) -> GND
- C12 pad 2: Net-(C10-Pad2) -> GND
- Y2 pad 2: Net-(C10-Pad2) -> GND
Routing:
- net GND: track 52.4 -> 62.8 mm, vias 21 -> 23
- net Net-(C10-Pad2): track 7.56 -> 0.00 mm, vias 2 -> 0
Changed lines of the file:
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@@
 (kicad_pcb (version 4) (host pcbnew 4.0.7-e2-6376~58~ubuntu16.04.1)
   (general
-    (links 121)
-    (no_connects 1)
+    (links 122)
+    (no_connects 0)
     (area 89.535 13.97 202.565001 69.215001)
     (thickness 1.6)
     (drawings 21)
-    (tracks 538)
+    (tracks 543)
     (zones 0)
     (modules 51)
-    (nets 86)
+    (nets 85)
   )
   (page A4)
@@
   )
   (setup
-    (last_trace_width 0.254)
+    (last_trace_width 0.15)
     (user_trace_width 0.254)
     (user_trace_width 0.508)
@@
     (visible_elements FFFFFF7F)
     (pcbplotparams
-      (layerselection 0x00030_80000001)
+      (layerselection 0x010f0_80000001)
       (usegerberextensions false)
       (excludeedgelayer true)
@@
       (padsonsilk false)
       (subtractmaskfromsilk false)
-      (outputformat 1)
+      (outputformat 4)
       (mirror false)
-      (drillshape 1)
+      (drillshape 0)
       (scaleselection 1)
       (outputdirectory ""))
@@
   (net 83 "Net-(R16-Pad2)")
   (net 84 "Net-(R17-Pad2)")
-  (net 85 "Net-(C10-Pad2)")
   (net_class Default "This is the default net class."
     (clearance 0.15)
@@
     (add_net MOSI)
     (add_net MOSI_2)
-    (add_net "Net-(C10-Pad2)")
     (add_net "Net-(C11-Pad1)")
     (add_net "Net-(C13-Pad1)")
@@
       (net 10 XTAL2))
     (pad 2 smd rect (at 1 0 315) (size 1 1.25) (layers F.Cu F.Paste F.Mask)
-      (net 85 "Net-(C10-Pad2)"))
+      (net 2 GND))
     (model /home/josh/Formula/OEM_Preferred_Parts/3DModels/C_0805_OEM/C_0805.wrl
       (at (xyz 0 0 0))
@@
       (net 12 XTAL1))
     (pad 2 smd rect (at 1 0 45) (size 1 1.25) (layers F.Cu F.Paste F.Mask)
-      (net 85 "Net-(C10-Pad2)"))
+      (net 2 GND))
     (model /home/josh/Formula/OEM_Preferred_Parts/3DModels/C_0805_OEM/C_0805.wrl
       (at (xyz 0 0 0))
@@
       (net 12 XTAL1))
     (pad 2 smd rect (at 1.1 0.8 45) (size 1.4 1.2) (layers F.Cu F.Mask)
-      (net 85 "Net-(C10-Pad2)"))
+      (net 2 GND))
     (pad 3 smd rect (at 1.1 -0.8 45) (size 1.4 1.2) (layers F.Cu F.Mask)
       (net 10 XTAL2))
@@
     (effects (font (size 1.016 1.016) (thickness 0.1524)))
   )
-  (gr_text "328 Prog LEDs" (at 162.941 22.733 360) (layer F.SilkS)
+  (gr_text "328 Prog LEDs" (at 162.941 22.733) (layer F.SilkS)
     (effects (font (size 0.762 0.762) (thickness 0.1524)))
   )
@@
   (segment (start 168.007047 39.949639) (end 168.912793 39.043893) (width 0.254) (layer F.Cu) (net 1))
   (segment (start 168.912793 39.043893) (end 171.504893 39.043893) (width 0.254) (layer F.Cu) (net 1))
+  (segment (start 170.126503 34.839868) (end 169.177975 34.839868) (width 0.254) (layer F.Cu) (net 2))
+  (segment (start 169.177975 34.839868) (end 168.818589 35.199254) (width 0.254) (layer F.Cu) (net 2))
+  (segment (start 168.452903 35.199254) (end 168.388025 35.264132) (width 0.254) (layer F.Cu) (net 2))
+  (segment (start 168.818589 35.199254) (end 168.452903 35.199254) (width 0.254) (layer F.Cu) (net 2))
+  (segment (start 168.388025 35.264132) (end 167.439497 35.264132) (width 0.254) (layer F.Cu) (net 2))
+  (segment (start 123.19 35.306) (end 123.19 36.83) (width 0.762) (layer F.Cu) (net 2))
+  (via (at 123.19 36.83) (size 0.6) (drill 0.3) (layers F.Cu B.Cu) (net 2))
   (segment (start 136.144 39.54) (end 136.441 39.54) (width 0.254) (layer F.Cu) (net 2))
   (segment (start 136.441 39.54) (end 137.414 40.513) (width 0.254) (layer F.Cu) (net 2))
@@
   (segment (start 126.832 31.791) (end 127 31.623) (width 0.254) (layer F.Cu) (net 2))
   (via (at 127 31.623) (size 0.6) (drill 0.3) (layers F.Cu B.Cu) (net 2))
-  (segment (start 123.19 35.306) (end 123.19 36.83) (width 0.254) (layer F.Cu) (net 2))
-  (via (at 123.19 36.83) (size 0.6) (drill 0.3) (layers F.Cu B.Cu) (net 2))
   (segment (start 116.126 35.052) (end 115.697 35.052) (width 0.254) (layer F.Cu) (net 2))
   (segment (start 115.697 35.052) (end 114.935 34.29) (width 0.254) (layer F.Cu) (net 2))
@@
   (segment (start 150.948107 54.682107) (end 150.61595 54.682107) (width 0.254) (layer F.Cu) (net 2))
   (segment (start 150.61595 54.682107) (end 149.340703 55.957354) (width 0.254) (layer F.Cu) (net 2))
+  (segment (start 170.126503 34.839868) (end 170.519132 34.839868) (width 0.254) (layer F.Cu) (net 2))
+  (segment (start 170.519132 34.839868) (end 171.704 33.655) (width 0.254) (layer F.Cu) (net 2))
+  (segment (start 171.704 33.655) (end 171.311371 33.655) (width 0.254) (layer F.Cu) (net 2))
+  (segment (start 171.395107 36.108472) (end 170.126503 34.839868) (width 0.254) (layer F.Cu) (net 2))
+  (segment (start 171.395107 36.249893) (end 171.395107 36.108472) (width 0.254) (layer F.Cu) (net 2))
+  (segment (start 169.863571 35.1028) (end 170.126503 34.839868) (width 0.254) (layer F.Cu) (net 2))
+  (segment (start 171.395107 36.249893) (end 171.395107 36.267107) (width 0.254) (layer F.Cu) (net 2))
+  (segment (start 171.395107 36.267107) (end 172.339 37.211) (width 0.254) (layer F.Cu) (net 2))
+  (via (at 172.339 37.211) (size 0.6) (drill 0.3) (layers F.Cu B.Cu) (net 2))
+  (segment (start 171.704 33.655) (end 172.72 32.639) (width 0.254) (layer F.Cu) (net 2))
+  (via (at 172.72 32.639) (size 0.6) (drill 0.3) (layers F.Cu B.Cu) (net 2))
   (segment (start 147.431515 47.17682) (end 149.1722 45.436135) (width 0.254) (layer F.Cu) (net 3))
   (segment (start 149.1722 45.436135) (end 149.1722 44.574486) (width 0.254) (layer F.Cu) (net 3))
@@
   (segment (start 160.147 32.019) (end 161.371 30.795) (width 0.254) (layer F.Cu) (net 84))
   (segment (start 161.371 30.795) (end 161.671 30.795) (width 0.254) (layer F.Cu) (net 84))
-  (segment (start 170.126503 34.839868) (end 170.519132 34.839868) (width 0.254) (layer F.Cu) (net 85))
-  (segment (start 170.519132 34.839868) (end 171.704 33.655) (width 0.254) (layer F.Cu) (net 85))
-  (segment (start 171.704 33.655) (end 171.311371 33.655) (width 0.254) (layer F.Cu) (net 85))
-  (segment (start 171.395107 36.108472) (end 170.126503 34.839868) (width 0.254) (layer F.Cu) (net 85))
-  (segment (start 171.395107 36.249893) (end 171.395107 36.108472) (width 0.254) (layer F.Cu) (net 85))
-  (segment (start 169.863571 35.1028) (end 170.126503 34.839868) (width 0.254) (layer F.Cu) (net 85))
-  (segment (start 171.395107 36.249893) (end 171.395107 36.267107) (width 0.254) (layer F.Cu) (net 85))
-  (segment (start 171.395107 36.267107) (end 172.339 37.211) (width 0.254) (layer F.Cu) (net 85))
-  (via (at 172.339 37.211) (size 0.6) (drill 0.3) (layers F.Cu B.Cu) (net 85))
-  (segment (start 171.704 33.655) (end 172.72 32.639) (width 0.254) (layer F.Cu) (net 85))
-  (via (at 172.72 32.639) (size 0.6) (drill 0.3) (layers F.Cu B.Cu) (net 85))
   (zone (net 2) (net_name GND) (layer B.Cu) (hatch edge 0.508)
     (connect_pads (clearance 0.508))
