File: boards/charging/etc..kicad_pcb (KiCad board)
At the start: 2 copper layers, 70 x 70 mm, 49 parts, among them IC1 ATMEGA16M1, J1 interface, J2 LCD screen, P1 CONN_02X03, U1 TPS561201, U2 CAN_Transceiver, U3 CP2120, U4 LM3480, Y1 Crystal_SMD

Commit message: charging
Parts:
- removed D5: D_Zener_18V, footprints:DO-214AA
- removed D6: LED_0805, footprints:LED_0805_OEM
- removed R11: R_0_Jumper, footprints:R_2512_OEM
- removed R12: R_200, footprints:R_0805_OEM
- removed U3: CP2120, footprints:CP2120-QFN
- added C12: C_47uF, footprints:C_0805_OEM, F.Cu at (85.1, 121.9)
- added C13: C_22uF, footprints:C_0805_OEM, F.Cu at (76.2, 118.6)
- added D9: LED_0805, footprints:LED_0805_OEM, F.Cu at (159.9, 122.7)
- added P2: CONN_02X03, footprints:Pin_Header_Straight_2x03, F.Cu at (155.7, 103.3)
- added Y2: Crystal_SMD, footprints:Crystal_SMD_FA238, F.Cu at (166.7, 103.4)
- C10: value C_10uF -> C_0.1uF
- C11: value C_0.1uF -> C_1uF
- C2: value C_100pF -> C_0.1uF
- C3: value C_22uF -> C_100pF
- C6: value C_0.1uF -> C_30pF
- C7: value C_47uF -> C_30pF
- D7: value LED_0805 -> D_Zener_18V; footprint footprints:LED_0805_OEM -> footprints:DO-214AA
- J1: value interface -> LCD screen; footprint footprints:micromatch_female_ra_20 -> footprints:micromatch_female_vert_16
- J2: value LCD screen -> interface; footprint footprints:micromatch_female_ra_16 -> footprints:micromatch_female_vert_20
- R10: value R_55.1k -> R_200
- R13: value 4.7kR -> R_0_Jumper; footprint footprints:R_0805_OEM -> footprints:R_2512_OEM
- R14: value 4.7kR -> R_200
- R15: value 4.7kR -> R_55.1k
- R16, R17: value R_200 -> R_10k
- R18: value R_200 -> R_1k
- R2: value R_1k -> R_10k
- R9: value R_10k -> R_200
- RV1: value POT_TRIM -> POT_TRIM-device
- U1: value TPS561201 -> ATMEGA328P-AU; footprint footprints:SOT-23-6_OEM -> footprints:TQFP-32_7x7mm_Pitch0.8mm
- U4: value LM3480 -> TPS561201; footprint footprints:SOT-23F -> footprints:SOT-23-6_OEM
- moved F1 113.8 mm to (80.5, 130.8), turned to 0 degrees
- moved U4 109.2 mm to (70.9, 140.7)
- moved D7 107.4 mm to (72.6, 134.1)
- moved L1 107.2 mm to (81.0, 143.8)
- moved R17 102.1 mm to (72.9, 125.7)
- moved U1 101.9 mm to (100.6, 156.2), turned to 0 degrees
- moved R13 92.9 mm to (68.6, 113.8), turned to 0 degrees
- moved R16 91.6 mm to (66.5, 121.7)
- moved D8 91.4 mm to (81.3, 110.5), turned to 0 degrees
- moved C9 85.9 mm to (83.1, 125.2), turned to 0 degrees
- moved C10 85.2 mm to (82.0, 117.3)
- moved R15 76.7 mm to (78.8, 122.9), turned to 0 degrees
- moved R14 73.3 mm to (74.5, 108.2)
- moved U2 64.0 mm to (175.0, 152.9)
- moved C11 61.0 mm to (179.6, 134.3), turned to 0 degrees
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Connections:
- C10 pad 1: +3V3 -> Net-(C10-Pad1)
- C10 pad 2: GND -> Net-(C10-Pad2)
- C11 pad 1: +3V3 -> GND
- C11 pad 2: GND -> Net-(C11-Pad2)
- C2 pad 1: Net-(C2-Pad1) -> VCC
- C5 pad 1: Net-(C5-Pad1) -> XTAL2
- C6 pad 2: Net-(C6-Pad2) -> GND
- C7 pad 1: Net-(C7-Pad1) -> XTAL1
- C9 pad 1: VCC -> GND
- C9 pad 2: GND -> Net-(C11-Pad2)
- D7 pad 1: GND -> +12V
- D7 pad 2: Net-(D7-Pad2) -> GND
- F1 pad 2: Net-(C3-Pad1) -> Net-(C13-Pad1)
- IC1 pad 10: Net-(C5-Pad1) -> Net-(C6-Pad1)
- IC1 pad 13: CS -> Net-(IC1-Pad13)
- IC1 pad 16: Net-(IC1-Pad16) -> DATA
- IC1 pad 19: Net-(C2-Pad1) -> Net-(C3-Pad1)
- J1 pad 10: LED1 -> DB3
- J1 pad 11: LED2 -> DB4
- J1 pad 12: IMD -> DB5
- J1 pad 13: GND -> DB6
- J1 pad 14: AMS -> DB7
- J1 pad 15: GND -> VCC
- J1 pad 16: SDA -> GND
- J1 pad 17: SCL -> (no net)
- J1 pad 2: +12V -> VCC
- J1 pad 3: VCC -> Net-(J1-Pad3)
- J1 pad 4: MOSI -> RS
- J1 pad 5: MISO -> R/W
- J1 pad 6: SCK -> E
- J1 pad 7: RESET -> DB0
- J1 pad 8: CANH -> DB1
- J1 pad 9: CANL -> DB2
- J2 pad 10: DB3 -> LED1
- J2 pad 11: DB4 -> LED2
- J2 pad 12: DB5 -> IMD
- J2 pad 13: DB6 -> GND
- J2 pad 14: DB7 -> AMS
- J2 pad 15: VCC -> GND
- J2 pad 16: GND -> SDA
- J2 pad 2: VCC -> +12V
- J2 pad 3: Net-(J2-Pad3) -> VCC
- J2 pad 4: RS -> MOSI
- J2 pad 5: R/W -> MISO
- J2 pad 6: E -> SCK
- J2 pad 7: DB0 -> RESET
- J2 pad 8: DB1 -> CANH
- J2 pad 9: DB2 -> CANL
- L1 pad 1: Net-(C6-Pad2) -> Net-(C10-Pad2)
- L1 pad 2: Net-(C7-Pad1) -> Net-(C11-Pad2)
- P1 pad 5: RESET -> RST32
- R1 pad 2: Net-(C2-Pad1) -> Net-(C3-Pad1)
- R10 pad 1: Net-(R10-Pad1) -> LED5
- R10 pad 2: Net-(C7-Pad1) -> Net-(D4-Pad2)
- R13 pad 1: +3V3 -> VCC
- R13 pad 2: RST -> Net-(C11-Pad2)
- R14 pad 1: +3V3 -> VCC
- R14 pad 2: SCL -> Net-(D8-Pad2)
- R15 pad 1: +3V3 -> Net-(R15-Pad1)
- R15 pad 2: SDA -> Net-(C11-Pad2)
- R16 pad 1: GPIO_0 -> Net-(C13-Pad1)
- R16 pad 2: Net-(D6-Pad2) -> Net-(R16-Pad2)
- R17 pad 1: VCC -> Net-(R15-Pad1)
- R17 pad 2: Net-(D7-Pad2) -> GND
- R18 pad 1: +3V3 -> Net-(C13-Pad1)
- R18 pad 2: Net-(D8-Pad2) -> Net-(D9-Pad2)
- R2 pad 1: Net-(C3-Pad1) -> VCC
- R2 pad 2: Net-(D1-Pad2) -> RST32
- R3 pad 1: Net-(C3-Pad1) -> DATA
- R3 pad 2: Net-(R3-Pad2) -> VCC
- R4 pad 1: Net-(D3-Pad2) -> Net-(D2-Pad2)
- R5 pad 1: Net-(D2-Pad2) -> Net-(D1-Pad2)
- R9 pad 1: Net-(R10-Pad1) -> LED6
- R9 pad 2: GND -> Net-(D3-Pad2)
- RV1 pad 2: Net-(J2-Pad3) -> Net-(J1-Pad3)
- U1 pad 1: GND -> Net-(U1-Pad1)
- U1 pad 2: Net-(C6-Pad2) -> Net-(U1-Pad2)
- U1 pad 3: Net-(C3-Pad1) -> GND
- U1 pad 4: Net-(R10-Pad1) -> VCC
- U1 pad 5: Net-(R3-Pad2) -> GND
- U1 pad 6: Net-(C6-Pad1) -> VCC
- U4 pad 1: +3V3 -> GND
- U4 pad 2: VCC -> Net-(C10-Pad2)
- U4 pad 3: GND -> Net-(C13-Pad1)
- Y1 pad 3: Net-(C5-Pad1) -> Net-(C6-Pad1)
Routing:
- net SCK: track 121.4 -> 0.00 mm, vias 8 -> 0
- net +3V3: track 119.2 -> 0.00 mm, vias 14 -> 0
- net VCC: track 118.6 -> 0.00 mm, vias 11 -> 0
- net MISO: track 58.4 -> 0.00 mm
- net GND: track 56.1 -> 0.00 mm, vias 23 -> 0
- net RESET: track 54.0 -> 0.00 mm
- net MOSI: track 53.3 -> 0.00 mm
- net IMD: track 43.5 -> 0.00 mm
- net AMS: track 40.1 -> 0.00 mm
- net Net-(C3-Pad1): track 32.7 -> 0.00 mm, vias 2 -> 0
- net Net-(R10-Pad1): track 27.4 -> 0.00 mm
- net CS: track 24.3 -> 0.00 mm
- net +12V: track 24.0 -> 0.00 mm
- net LED2: track 22.2 -> 0.00 mm, vias 2 -> 0
- net RST: track 21.6 -> 0.00 mm
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- removed copper zone on B.Cu, net GND
Other:
- board outline removed

Commit message: Final charging with gerber
Parts:
- added J3: Ultrafit_4, footprints:Ultrafit_4, F.Cu at (131.4, 64.9)
- added J4: Ultrafit_4, footprints:Ultrafit_4, F.Cu at (157.3, 36.5)
- added U3: RJ45_VT, footprints:RJ45-Vertical, F.Cu at (117.9, 31.7)
- J2: value interface -> Ampseal_8; footprint footprints:micromatch_female_vert_20 -> footprints:Ampseal_8
- RV1: footprint footprints:Potentiometer_Trimmer_Bourns_TC33X-1 -> footprints:Potentiometer_Trimmer_Bourns_TCC3
- moved U1 130.8 mm to (147.9, 34.2), turned to 270 degrees
- moved U2 107.9 mm to (131.4, 54.3), turned to 270 degrees
- moved R6 107.7 mm to (131.1, 42.1), turned to 90 degrees
- moved C7 106.2 mm to (136.7, 34.2), turned to 270 degrees
- moved C11 104.6 mm to (100.8, 65.6), turned to 270 degrees
- moved C5 101.8 mm to (140.5, 33.7), turned to 180 degrees
- moved R5 99.6 mm to (134.4, 47.2), turned to 315 degrees
- moved R10 98.9 mm to (146.9, 41.6), turned to 270 degrees
- moved R7 97.7 mm to (122.0, 48.9)
- moved R8 93.7 mm to (125.5, 48.9)
- moved RV1 93.5 mm to (154.7, 49.5), turned to 270 degrees
- moved D4 91.0 mm to (147.5, 44.4), turned to 180 degrees
- moved P1 90.8 mm to (133.6, 35.5), turned to 180 degrees
- moved R2 89.5 mm to (151.7, 40.8)
- moved R14 87.5 mm to (149.2, 62.7), turned to 180 degrees
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Connections:
- J2 pad 2: +12V -> GND
- J2 pad 3: VCC -> +12V
- J2 pad 4: MOSI -> CANH
- J2 pad 5: MISO -> +12V
- J2 pad 6: SCK -> CANH
- J2 pad 7: RESET -> CANL
- J2 pad 8: CANH -> CANL
Routing:
- net VCC: track 0.00 -> 207.2 mm, vias 0 -> 10
- net GND: track 0.00 -> 102.4 mm, vias 0 -> 24
- net SCK: track 0.00 -> 82.5 mm, vias 0 -> 4
- net CANH: track 0.00 -> 68.4 mm
- net CANL: track 0.00 -> 53.4 mm
- net RST32: track 0.00 -> 50.7 mm
- net +12V: track 0.00 -> 46.2 mm
- net MOSI: track 0.00 -> 44.3 mm, vias 0 -> 2
- net MISO: track 0.00 -> 40.9 mm
- net RESET: track 0.00 -> 37.4 mm, vias 0 -> 5
- net DATA: track 0.00 -> 27.4 mm, vias 0 -> 6
- net Net-(C11-Pad2): track 0.00 -> 27.0 mm
- net DB7: track 0.00 -> 23.5 mm
- net RS: track 0.00 -> 23.2 mm
- net LED2: track 0.00 -> 22.0 mm
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- added copper zone on B.Cu, net GND
Other:
- board outline added: 97 x 64 mm
- net class Default: trace_width 0.25 -> 0.254
- rule pad_to_mask_clearance: 0.2 -> 0
- rule trace_min: 0.254 -> 0.1524

Commit message: Charging w Gerber checked off
Parts:
- C13: footprint footprints:C_0805_OEM -> footprints:C_1206_OEM
Routing:
- net Net-(C13-Pad1): track 21.4 -> 17.4 mm
Other:
- outline, holes or cut-outs redrawn
- board text added: "12 V"
- board text added: "5V"
- board text added: "Olin Electric Motorsports Hyegi Bang Charging v1 3.09.2018"
