File: boards/charging/etc..sch (KiCad schematic (older format))
At the start: 49 parts, among them IC1 ATMEGA16M1, J1 interface, J2 LCD screen, P1 CONN_02X03, U1 TPS561201, U2 CAN_Transceiver, U3 CP2120, U4 LM3480, Y1 Crystal_SMD

Commit message: charging
Parts:
- removed C10: C_10uF, footprints:C_0805_OEM, symbol C_10uF
- removed C11, C9: C_0.1uF, footprints:C_0805_OEM, symbol C_0.1uF
- removed D6, D7, D8: LED_0805, footprints:LED_0805_OEM, symbol LED_0805
- removed J1: interface, footprints:micromatch_female_ra_20, symbol micromatch_male_20
- removed R13, R14, R15: 4.7kR, footprints:R_0805_OEM, symbol 4.7kR
- removed R16, R17, R18: R_200, footprints:R_0805_OEM, symbol R_200
- removed RV1: POT_TRIM, footprints:Potentiometer_Trimmer_Bourns_TC33X-1, symbol POT_TRIM
- removed U3: CP2120, footprints:CP2120-QFN, symbol CP2120
- removed U4: LM3480, footprints:SOT-23F, symbol LM3480
- added C1, C9: C_0.1uF, footprints:C_0805_OEM, symbol etc.-rescue:C_0.1uF-formula
- added C11: C_1uF, footprints:C_0805_OEM, symbol etc.-rescue:C_1uF-formula
- added C5, C7: C_30pF, footprints:C_0805_OEM, symbol etc.-rescue:C_30pF-formula
- added D3, D4: LED_0805, footprints:LED_0805_OEM, symbol etc.-rescue:LED_0805-formula
- added J2: Ampseal_8, symbol formula:Ampseal_8
- added J3, J4: Ultrafit_4, footprints:Ultrafit_4, symbol formula:Ultrafit_4
- added P1: CONN_02X03, footprints:Pin_Header_Straight_2x03, symbol etc.-rescue:CONN_02X03-formula
- added R10, R9: R_200, footprints:R_0805_OEM, symbol etc.-rescue:R_200-formula
- added R2, R3: R_10k, footprints:R_0805_OEM, symbol etc.-rescue:R_10k-formula
- added RV1: POT_TRIM-device, footprints:Potentiometer_Trimmer_Bourns_TC33X-1, symbol etc.-rescue:POT_TRIM-device
- added U1: ATMEGA328P-AU, footprints:TQFP-32_7x7mm_Pitch0.8mm, symbol etc.-rescue:ATMEGA328P-AU-atmel
- added U3: RJ45_VT, footprints:RJ45-Vertical, symbol formula:RJ45_VT
- added Y2: Crystal_SMD, footprints:Crystal_SMD_FA238, symbol etc.-rescue:Crystal_SMD-formula
- C10: renamed from C6; symbol C_0.1uF -> etc.-rescue:C_0.1uF-formula
- C12: renamed from C7; symbol C_47uF -> etc.-rescue:C_47uF-formula
- C13: renamed from C3; symbol C_22uF -> etc.-rescue:C_22uF-formula
- C2: renamed from C1; symbol C_0.1uF -> etc.-rescue:C_0.1uF-formula
- C3: renamed from C2; symbol C_100pF -> etc.-rescue:C_100pF-formula
- C4: symbol C_30pF -> etc.-rescue:C_30pF-formula
- C6: renamed from C5; symbol C_30pF -> etc.-rescue:C_30pF-formula
- C8: symbol C_0.1uF -> etc.-rescue:C_0.1uF-formula
- D1: renamed from D2; symbol LED_0805 -> etc.-rescue:LED_0805-formula
- D2: renamed from D3; symbol LED_0805 -> etc.-rescue:LED_0805-formula
- D7: renamed from D5; symbol D_Zener_18V -> etc.-rescue:D_Zener_18V-formula
- D8: renamed from D4; symbol LED_0805 -> etc.-rescue:LED_0805-formula
- D9: renamed from D1; symbol LED_0805 -> etc.-rescue:LED_0805-formula
- F1: symbol F_500mA_16V -> etc.-rescue:F_500mA_16V-formula
- IC1: symbol ATMEGA16M1 -> etc.-rescue:ATMEGA16M1-formula
- J1: renamed from J2; footprint footprints:micromatch_female_ra_16 -> footprints:micromatch_female_vert_16; symbol micromatch_male_16 -> etc.-rescue:micromatch_male_16-formula
- L1: symbol L_4.7uH -> etc.-rescue:L_4.7uH-formula
- P2: renamed from P1; symbol CONN_02X03 -> etc.-rescue:CONN_02X03-formula
- R1: symbol R_100 -> etc.-rescue:R_100-formula
- R13: renamed from R11; symbol R_0_Jumper -> etc.-rescue:R_0_Jumper-formula
- R14: renamed from R12; symbol R_200 -> etc.-rescue:R_200-formula
- R15: renamed from R10; symbol R_55.1k -> etc.-rescue:R_55.1k-formula
- R16: renamed from R3; symbol R_10k -> etc.-rescue:R_10k-formula
- R17: renamed from R9; symbol R_10k -> etc.-rescue:R_10k-formula
- R18: renamed from R2; symbol R_1k -> etc.-rescue:R_1k-formula
- R4, R5, R7, R8: symbol R_200 -> etc.-rescue:R_200-formula
- R6: symbol R_10k -> etc.-rescue:R_10k-formula
- U2: symbol CAN_Transceiver -> etc.-rescue:CAN_Transceiver-formula
- U4: renamed from U1; symbol TPS561201 -> etc.-rescue:TPS561201-formula
- Y1: symbol Crystal_SMD -> etc.-rescue:Crystal_SMD-formula
Connections:
- net labels added: DATA, LED5, LED6, RST32, XTAL1, XTAL2
- net labels removed: +3.3V, CS, EINT, GPIO_0, INT, RST
- wire segments 72 -> 90
- no-connect marks 12 -> 18

Commit message: Final charging with gerber
Parts:
- C1, C10, C2, C8, C9: symbol etc.-rescue:C_0.1uF-formula -> etc.-rescue:C_0.1uF-formula-etc.-rescue-etc.-rescue
- C11: symbol etc.-rescue:C_1uF-formula -> etc.-rescue:C_1uF-formula-etc.-rescue-etc.-rescue
- C12: symbol etc.-rescue:C_47uF-formula -> etc.-rescue:C_47uF-formula-etc.-rescue-etc.-rescue
- C13: symbol etc.-rescue:C_22uF-formula -> etc.-rescue:C_22uF-formula-etc.-rescue-etc.-rescue
- C3: symbol etc.-rescue:C_100pF-formula -> etc.-rescue:C_100pF-formula-etc.-rescue-etc.-rescue
- C4, C5, C6, C7: symbol etc.-rescue:C_30pF-formula -> etc.-rescue:C_30pF-formula-etc.-rescue-etc.-rescue
- D1, D2, D3, D4, D8, D9: symbol etc.-rescue:LED_0805-formula -> etc.-rescue:LED_0805-formula-etc.-rescue-etc.-rescue
- D7: symbol etc.-rescue:D_Zener_18V-formula -> etc.-rescue:D_Zener_18V-formula-etc.-rescue-etc.-rescue
- F1: symbol etc.-rescue:F_500mA_16V-formula -> etc.-rescue:F_500mA_16V-formula-etc.-rescue-etc.-rescue
- IC1: symbol etc.-rescue:ATMEGA16M1-formula -> etc.-rescue:ATMEGA16M1-formula-etc.-rescue-etc.-rescue
- J1: symbol etc.-rescue:micromatch_male_16-formula -> etc.-rescue:micromatch_male_16-formula-etc.-rescue-etc.-rescue
- J2: footprint (none) -> footprints:Ampseal_8
- L1: symbol etc.-rescue:L_4.7uH-formula -> etc.-rescue:L_4.7uH-formula-etc.-rescue-etc.-rescue
- P1, P2: symbol etc.-rescue:CONN_02X03-formula -> etc.-rescue:CONN_02X03-formula-etc.-rescue-etc.-rescue
- R1: symbol etc.-rescue:R_100-formula -> etc.-rescue:R_100-formula-etc.-rescue-etc.-rescue
- R10, R14, R4, R5, R7, R8, R9: symbol etc.-rescue:R_200-formula -> etc.-rescue:R_200-formula-etc.-rescue-etc.-rescue
- R13: symbol etc.-rescue:R_0_Jumper-formula -> etc.-rescue:R_0_Jumper-formula-etc.-rescue-etc.-rescue
- R15: symbol etc.-rescue:R_55.1k-formula -> etc.-rescue:R_55.1k-formula-etc.-rescue-etc.-rescue
- R16, R17, R2, R3, R6: symbol etc.-rescue:R_10k-formula -> etc.-rescue:R_10k-formula-etc.-rescue-etc.-rescue
- R18: symbol etc.-rescue:R_1k-formula -> etc.-rescue:R_1k-formula-etc.-rescue-etc.-rescue
- RV1: footprint footprints:Potentiometer_Trimmer_Bourns_TC33X-1 -> footprints:Potentiometer_Trimmer_Bourns_TCC3; symbol etc.-rescue:POT_TRIM-device -> etc.-rescue:POT_TRIM-device-etc.-rescue-etc.-rescue
- U1: symbol etc.-rescue:ATMEGA328P-AU-atmel -> etc.-rescue:ATMEGA328P-AU-atmel-etc.-rescue-etc.-rescue
- U2: symbol etc.-rescue:CAN_Transceiver-formula -> etc.-rescue:CAN_Transceiver-formula-etc.-rescue-etc.-rescue
- U4: symbol etc.-rescue:TPS561201-formula -> etc.-rescue:TPS561201-formula-etc.-rescue-etc.-rescue
- Y1, Y2: symbol etc.-rescue:Crystal_SMD-formula -> etc.-rescue:Crystal_SMD-formula-etc.-rescue-etc.-rescue
Connections:
- wire segments 90 -> 105

Commit message: Charging w Gerber checked off
Parts:
- C1, C10, C2, C8, C9: symbol etc.-rescue:C_0.1uF-formula-etc.-rescue-etc.-rescue -> etc.-rescue:C_0.1uF-formula-etc.-rescue-etc.-rescue-etc.-rescue
- C11: symbol etc.-rescue:C_1uF-formula-etc.-rescue-etc.-rescue -> etc.-rescue:C_1uF-formula-etc.-rescue-etc.-rescue-etc.-rescue
- C12: symbol etc.-rescue:C_47uF-formula-etc.-rescue-etc.-rescue -> etc.-rescue:C_47uF-formula-etc.-rescue-etc.-rescue-etc.-rescue
- C13: footprint footprints:C_0805_OEM -> footprints:C_1206_OEM; symbol etc.-rescue:C_22uF-formula-etc.-rescue-etc.-rescue -> etc.-rescue:C_22uF-formula-etc.-rescue-etc.-rescue-etc.-rescue
- C3: symbol etc.-rescue:C_100pF-formula-etc.-rescue-etc.-rescue -> etc.-rescue:C_100pF-formula-etc.-rescue-etc.-rescue-etc.-rescue
- C4, C5, C6, C7: symbol etc.-rescue:C_30pF-formula-etc.-rescue-etc.-rescue -> etc.-rescue:C_30pF-formula-etc.-rescue-etc.-rescue-etc.-rescue
- D1, D2, D3, D4, D8, D9: symbol etc.-rescue:LED_0805-formula-etc.-rescue-etc.-rescue -> etc.-rescue:LED_0805-formula-etc.-rescue-etc.-rescue-etc.-rescue
- D7: symbol etc.-rescue:D_Zener_18V-formula-etc.-rescue-etc.-rescue -> etc.-rescue:D_Zener_18V-formula-etc.-rescue-etc.-rescue-etc.-rescue
- F1: symbol etc.-rescue:F_500mA_16V-formula-etc.-rescue-etc.-rescue -> etc.-rescue:F_500mA_16V-formula-etc.-rescue-etc.-rescue-etc.-rescue
- IC1: symbol etc.-rescue:ATMEGA16M1-formula-etc.-rescue-etc.-rescue -> etc.-rescue:ATMEGA16M1-formula-etc.-rescue-etc.-rescue-etc.-rescue
- J1: symbol etc.-rescue:micromatch_male_16-formula-etc.-rescue-etc.-rescue -> etc.-rescue:micromatch_male_16-formula-etc.-rescue-etc.-rescue-etc.-rescue
- L1: symbol etc.-rescue:L_4.7uH-formula-etc.-rescue-etc.-rescue -> etc.-rescue:L_4.7uH-formula-etc.-rescue-etc.-rescue-etc.-rescue
- P1, P2: symbol etc.-rescue:CONN_02X03-formula-etc.-rescue-etc.-rescue -> etc.-rescue:CONN_02X03-formula-etc.-rescue-etc.-rescue-etc.-rescue
- R1: symbol etc.-rescue:R_100-formula-etc.-rescue-etc.-rescue -> etc.-rescue:R_100-formula-etc.-rescue-etc.-rescue-etc.-rescue
- R10, R14, R4, R5, R7, R8, R9: symbol etc.-rescue:R_200-formula-etc.-rescue-etc.-rescue -> etc.-rescue:R_200-formula-etc.-rescue-etc.-rescue-etc.-rescue
- R13: symbol etc.-rescue:R_0_Jumper-formula-etc.-rescue-etc.-rescue -> etc.-rescue:R_0_Jumper-formula-etc.-rescue-etc.-rescue-etc.-rescue
- R15: symbol etc.-rescue:R_55.1k-formula-etc.-rescue-etc.-rescue -> etc.-rescue:R_55.1k-formula-etc.-rescue-etc.-rescue-etc.-rescue
- R16, R17, R2, R3, R6: symbol etc.-rescue:R_10k-formula-etc.-rescue-etc.-rescue -> etc.-rescue:R_10k-formula-etc.-rescue-etc.-rescue-etc.-rescue
- R18: symbol etc.-rescue:R_1k-formula-etc.-rescue-etc.-rescue -> etc.-rescue:R_1k-formula-etc.-rescue-etc.-rescue-etc.-rescue
- RV1: symbol etc.-rescue:POT_TRIM-device-etc.-rescue-etc.-rescue -> etc.-rescue:POT_TRIM-device-etc.-rescue-etc.-rescue-etc.-rescue
- U1: symbol etc.-rescue:ATMEGA328P-AU-atmel-etc.-rescue-etc.-rescue -> etc.-rescue:ATMEGA328P-AU-atmel-etc.-rescue-etc.-rescue-etc.-rescue
- U2: symbol etc.-rescue:CAN_Transceiver-formula-etc.-rescue-etc.-rescue -> etc.-rescue:CAN_Transceiver-formula-etc.-rescue-etc.-rescue-etc.-rescue
- U4: symbol etc.-rescue:TPS561201-formula-etc.-rescue-etc.-rescue -> etc.-rescue:TPS561201-formula-etc.-rescue-etc.-rescue-etc.-rescue
- Y1, Y2: symbol etc.-rescue:Crystal_SMD-formula-etc.-rescue-etc.-rescue -> etc.-rescue:Crystal_SMD-formula-etc.-rescue-etc.-rescue-etc.-rescue
Changed lines of the file:
@@
 $EndDescr
 $Comp
-L etc.-rescue:R_10k-formula-etc.-rescue-etc.-rescue R16
+L etc.-rescue:R_10k-formula-etc.-rescue-etc.-rescue-etc.-rescue R16
 U 1 1 59E042A3
 P 9700 5450
@@
 $EndComp
 $Comp
-L etc.-rescue:R_10k-formula-etc.-rescue-etc.-rescue R17
+L etc.-rescue:R_10k-formula-etc.-rescue-etc.-rescue-etc.-rescue R17
 U 1 1 59E042EA
 P 9850 4400
@@
 $EndComp
 $Comp
-L etc.-rescue:R_1k-formula-etc.-rescue-etc.-rescue R18
+L etc.-rescue:R_1k-formula-etc.-rescue-etc.-rescue-etc.-rescue R18
 U 1 1 59E0432B
 P 9850 5950
@@
 $EndComp
 $Comp
-L etc.-rescue:R_55.1k-formula-etc.-rescue-etc.-rescue R15
+L etc.-rescue:R_55.1k-formula-etc.-rescue-etc.-rescue-etc.-rescue R15
 U 1 1 59E0438C
 P 9700 4200
@@
 $EndComp
 $Comp
-L etc.-rescue:R_200-formula-etc.-rescue-etc.-rescue R14
+L etc.-rescue:R_200-formula-etc.-rescue-etc.-rescue-etc.-rescue R14
 U 1 1 59E04401
 P 9650 3150
@@
 $EndComp
 $Comp
-L etc.-rescue:R_0_Jumper-formula-etc.-rescue-etc.-rescue R13
+L etc.-rescue:R_0_Jumper-formula-etc.-rescue-etc.-rescue-etc.-rescue R13
 U 1 1 59E0444E
 P 9500 3500
@@
 $EndComp
 $Comp
-L etc.-rescue:LED_0805-formula-etc.-rescue-etc.-rescue D9
+L etc.-rescue:LED_0805-formula-etc.-rescue-etc.-rescue-etc.-rescue D9
 U 1 1 59E047E3
 P 10150 5950
@@
 $EndComp
 $Comp
-L etc.-rescue:LED_0805-formula-etc.-rescue-etc.-rescue D8
+L etc.-rescue:LED_0805-formula-etc.-rescue-etc.-rescue-etc.-rescue D8
 U 1 1 59E0483A
 P 9950 3150
@@
 $EndComp
 $Comp
-L etc.-rescue:L_4.7uH-formula-etc.-rescue-etc.-rescue L1
+L etc.-rescue:L_4.7uH-formula-etc.-rescue-etc.-rescue-etc.-rescue L1
 U 1 1 59E04875
 P 9500 3850
@@
 $EndComp
 $Comp
-L etc.-rescue:C_0.1uF-formula-etc.-rescue-etc.-rescue C10
+L etc.-rescue:C_0.1uF-formula-etc.-rescue-etc.-rescue-etc.-rescue C10
 U 1 1 59E048C8
 P 9350 4250
@@
 $EndComp
 $Comp
-L etc.-rescue:C_22uF-formula-etc.-rescue-etc.-rescue C13
+L etc.-rescue:C_22uF-formula-etc.-rescue-etc.-rescue-etc.-rescue C13
 U 1 1 59E04907
 P 9850 5700
 F 0 "C13" H 9875 5800 50  0000 L CNN
 F 1 "C_22uF" H 9875 5600 50  0000 L CNN
-F 2 "footprints:C_0805_OEM" H 9888 5550 50  0001 C CNN
+F 2 "footprints:C_1206_OEM" H 9888 5550 50  0001 C CNN
 F 3 "http://www.samsungsem.com/kr/support/product-search/mlcc/__icsFiles/afieldfile/2017/07/28/S_CL31A226KOCLFNC.pdf" H 9875 5800 50  0001 C CNN
 F 4 "1276-2725-1-ND" H 9850 5700 60  0001 C CNN "MPN"
@@
 $EndComp
 $Comp
-L etc.-rescue:C_47uF-formula-etc.-rescue-etc.-rescue C12
+L etc.-rescue:C_47uF-formula-etc.-rescue-etc.-rescue-etc.-rescue C12
 U 1 1 59E0494E
 P 9850 3650
@@
 $EndComp
 $Comp
-L etc.-rescue:TPS561201-formula-etc.-rescue-etc.-rescue U4
+L etc.-rescue:TPS561201-formula-etc.-rescue-etc.-rescue-etc.-rescue U4
 U 1 1 59E04993
 P 9600 4850
@@
 $EndComp
 $Comp
-L etc.-rescue:F_500mA_16V-formula-etc.-rescue-etc.-rescue F1
+L etc.-rescue:F_500mA_16V-formula-etc.-rescue-etc.-rescue-etc.-rescue F1
 U 1 1 59E0A5CF
 P 9550 5950
@@
 $EndComp
 $Comp
-L etc.-rescue:R_100-formula-etc.-rescue-etc.-rescue R1
+L etc.-rescue:R_100-formula-etc.-rescue-etc.-rescue-etc.-rescue R1
 U 1 1 59E06840
 P 1950 1450
@@
 $EndComp
 $Comp
-L etc.-rescue:C_0.1uF-formula-etc.-rescue-etc.-rescue C8
+L etc.-rescue:C_0.1uF-formula-etc.-rescue-etc.-rescue-etc.-rescue C8
 U 1 1 59E068FA
 P 6450 2150
@@
 $EndComp
 $Comp
-L etc.-rescue:C_0.1uF-formula-etc.-rescue-etc.-rescue C2
+L etc.-rescue:C_0.1uF-formula-etc.-rescue-etc.-rescue-etc.-rescue C2
 U 1 1 59E06957
 P 1750 1450
@@
 $EndComp
 $Comp
-L etc.-rescue:C_100pF-formula-etc.-rescue-etc.-rescue C3
+L etc.-rescue:C_100pF-formula-etc.-rescue-etc.-rescue-etc.-rescue C3
 U 1 1 59E06E67
 P 1950 1750
@@
 $EndComp
 $Comp
-L etc.-rescue:C_30pF-formula-etc.-rescue-etc.-rescue C6
+L etc.-rescue:C_30pF-formula-etc.-rescue-etc.-rescue-etc.-rescue C6
 U 1 1 59E06ED0
 P 4650 4450
@@
 $EndComp
 $Comp
-L etc.-rescue:C_30pF-formula-etc.-rescue-etc.-rescue C4
+L etc.-rescue:C_30pF-formula-etc.-rescue-etc.-rescue-etc.-rescue C4
 U 1 1 59E06F43
 P 4350 4450
@@
 $EndComp
 $Comp
-L etc.-rescue:R_10k-formula-etc.-rescue-etc.-rescue R6
+L etc.-rescue:R_10k-formula-etc.-rescue-etc.-rescue-etc.-rescue R6
 U 1 1 59E087A5
 P 4750 3850
@@
 RXCAN
 $Comp
-L etc.-rescue:ATMEGA16M1-formula-etc.-rescue-etc.-rescue IC1
+L etc.-rescue:ATMEGA16M1-formula-etc.-rescue-etc.-rescue-etc.-rescue IC1
 U 1 1 59E10948
 P 3250 3000
@@
 $EndComp
 $Comp
-L etc.-rescue:Crystal_SMD-formula-etc.-rescue-etc.-rescue Y1
+L etc.-rescue:Crystal_SMD-formula-etc.-rescue-etc.-rescue-etc.-rescue Y1
 U 1 1 59E10C38
 P 4500 4300
@@
 $EndComp
 $Comp
-L etc.-rescue:CONN_02X03-formula-etc.-rescue-etc.-rescue P2
+L etc.-rescue:CONN_02X03-formula-etc.-rescue-etc.-rescue-etc.-rescue P2
 U 1 1 59E10F9E
 P 5350 3400
@@
 $EndComp
 $Comp
-L etc.-rescue:CAN_Transceiver-formula-etc.-rescue-etc.-rescue U2
+L etc.-rescue:CAN_Transceiver-formula-etc.-rescue-etc.-rescue-etc.-rescue U2
 U 1 1 59E1176B
 P 6300 2600
@@
 DB7
 $Comp
-L etc.-rescue:R_200-formula-etc.-rescue-etc.-rescue R4
+L etc.-rescue:R_200-formula-etc.-rescue-etc.-rescue-etc.-rescue R4
 U 1 1 59E889C3
 P 4700 2600
@@
 $EndComp
 $Comp
-L etc.-rescue:R_200-formula-etc.-rescue-etc.-rescue R5
+L etc.-rescue:R_200-formula-etc.-rescue-etc.-rescue-etc.-rescue R5
 U 1 1 59E88C19
 P 4750 2300
@@
 $EndComp
 $Comp
-L etc.-rescue:LED_0805-formula-etc.-rescue-etc.-rescue D1
+L etc.-rescue:LED_0805-formula-etc.-rescue-etc.-rescue-etc.-rescue D1
 U 1 1 59E8C0F2
 P 5200 2300
@@
 $EndComp
 $Comp
-L etc.-rescue:LED_0805-formula-etc.-rescue-etc.-rescue D2
+L etc.-rescue:LED_0805-formula-etc.-rescue-etc.-rescue-etc.-rescue D2
 U 1 1 59E8C23B
 P 5200 2600
@@
 $EndComp
 $Comp
-L etc.-rescue:R_200-formula-etc.-rescue-etc.-rescue R7
+L etc.-rescue:R_200-formula-etc.-rescue-etc.-rescue-etc.-rescue R7
 U 1 1 59E95678
 P 4900 1400
@@
 $EndComp
 $Comp
-L etc.-rescue:R_200-formula-etc.-rescue-etc.-rescue R8
+L etc.-rescue:R_200-formula-etc.-rescue-etc.-rescue-etc.-rescue R8
 U 1 1 59E959F8
 P 4950 1300
@@
 	9400 5700 9700 5700
 $Comp
-L etc.-rescue:D_Zener_18V-formula-etc.-rescue-etc.-rescue D7
+L etc.-rescue:D_Zener_18V-formula-etc.-rescue-etc.-rescue-etc.-rescue D7
 U 1 1 5A00A462
 P 9600 6450
@@
 	2150 3800 2150 4200
 $Comp
-L etc.-rescue:ATMEGA328P-AU-atmel-etc.-rescue-etc.-rescue U1
+L etc.-rescue:ATMEGA328P-AU-atmel-etc.-rescue-etc.-rescue-etc.-rescue U1
 U 1 1 5A7A32AF
 P 2350 6250
@@
 NoConn ~ 1450 6600
 $Comp
-L etc.-rescue:C_0.1uF-formula-etc.-rescue-etc.-rescue C1
+L etc.-rescue:C_0.1uF-formula-etc.-rescue-etc.-rescue-etc.-rescue C1
 U 1 1 5A7BDCE5
 P 900 6250
@@
 	900  7350 1300 7350
 $Comp
-L etc.-rescue:R_10k-formula-etc.-rescue-etc.-rescue R3
+L etc.-rescue:R_10k-formula-etc.-rescue-etc.-rescue-etc.-rescue R3
 U 1 1 5A7D1C46
 P 4250 5150
@@
 	3350 6600 3900 6600
 $Comp
-L etc.-rescue:R_10k-formula-etc.-rescue-etc.-rescue R2
+L etc.-rescue:R_10k-formula-etc.-rescue-etc.-rescue-etc.-rescue R2
 U 1 1 5A7E5A0D
 P 3900 6450
@@
 RST32
 $Comp
-L etc.-rescue:CONN_02X03-formula-etc.-rescue-etc.-rescue P1
+L etc.-rescue:CONN_02X03-formula-etc.-rescue-etc.-rescue-etc.-rescue P1
 U 1 1 5A7EB2B5
 P 4400 7550
@@
 	4650 7650 4700 7650
 $Comp
-L etc.-rescue:R_200-formula-etc.-rescue-etc.-rescue R9
+L etc.-rescue:R_200-formula-etc.-rescue-etc.-rescue-etc.-rescue R9
 U 1 1 5A7ED913
 P 5500 5350
@@
 	5500 5500 5500 5650
 $Comp
-L etc.-rescue:LED_0805-formula-etc.-rescue-etc.-rescue D3
+L etc.-rescue:LED_0805-formula-etc.-rescue-etc.-rescue-etc.-rescue D3
 U 1 1 5A7ED920
 P 5500 5800
@@
 $EndComp
 $Comp
-L etc.-rescue:R_200-formula-etc.-rescue-etc.-rescue R10
+L etc.-rescue:R_200-formula-etc.-rescue-etc.-rescue-etc.-rescue R10
 U 1 1 5A7ED932
 P 5850 5350
@@
 	5850 5500 5850 5650
 $Comp
-L etc.-rescue:LED_0805-formula-etc.-rescue-etc.-rescue D4
+L etc.-rescue:LED_0805-formula-etc.-rescue-etc.-rescue-etc.-rescue D4
 U 1 1 5A7ED93F
 P 5850 5800
@@
 LED6
 $Comp
-L etc.-rescue:C_30pF-formula-etc.-rescue-etc.-rescue C7
+L etc.-rescue:C_30pF-formula-etc.-rescue-etc.-rescue-etc.-rescue C7
 U 1 1 5A7F36AA
 P 4750 6100
@@
 $EndComp
 $Comp
-L etc.-rescue:C_30pF-formula-etc.-rescue-etc.-rescue C5
+L etc.-rescue:C_30pF-formula-etc.-rescue-etc.-rescue-etc.-rescue C5
 U 1 1 5A7F36B5
 P 4450 6100
@@
 $EndComp
 $Comp
-L etc.-rescue:Crystal_SMD-formula-etc.-rescue-etc.-rescue Y2
+L etc.-rescue:Crystal_SMD-formula-etc.-rescue-etc.-rescue-etc.-rescue Y2
 U 1 1 5A7F36D9
 P 4600 5950
@@
 NoConn ~ 4350 3600
 $Comp
-L etc.-rescue:micromatch_male_16-formula-etc.-rescue-etc.-rescue J1
+L etc.-rescue:micromatch_male_16-formula-etc.-rescue-etc.-rescue-etc.-rescue J1
 U 1 1 59E83768
 P 7350 3600
@@
 	6800 4800 6800 4500
 $Comp
-L etc.-rescue:POT_TRIM-device-etc.-rescue-etc.-rescue RV1
+L etc.-rescue:POT_TRIM-device-etc.-rescue-etc.-rescue-etc.-rescue RV1
 U 1 1 5A97B362
 P 8550 3700
@@
 E
 $Comp
-L etc.-rescue:C_0.1uF-formula-etc.-rescue-etc.-rescue C9
+L etc.-rescue:C_0.1uF-formula-etc.-rescue-etc.-rescue-etc.-rescue C9
 U 1 1 5A98A088
 P 9850 3850
@@
 	9700 3850 9700 4000
 $Comp
-L etc.-rescue:C_1uF-formula-etc.-rescue-etc.-rescue C11
+L etc.-rescue:C_1uF-formula-etc.-rescue-etc.-rescue-etc.-rescue C11
 U 1 1 5A98A2D0
 P 10100 4000
@@
 	6800 4500 7200 4500
 $Comp
-L power:GND #PWR?
+L power:GND #PWR0117
 U 1 1 5AA25D47
 P 7700 6340
-F 0 "#PWR?" H 7700 6090 50  0001 C CNN
+F 0 "#PWR0117" H 7700 6090 50  0001 C CNN
 F 1 "GND" H 7705 6167 50  0000 C CNN
 F 2 "" H 7700 6340 50  0001 C CNN
