File: boards/dashboard/ExternalInterface/ExternalInterface.sch (KiCad schematic (older format))
At the start: 2 parts

Commit message: Boards updated
Parts:
- removed J?: micromatch_female_RA_14, footprints:micromatch_female_ra_14, symbol micromatch_female_RA_14
- added J1: micromatch_female_TOP_ENTRY_locking_14, footprints:micromatch_female_vert_14, symbol micromatch_female_TOP_ENTRY_locking_14
- added J3: micromatch_female_TOP_ENTRY_locking_6, footprints:micromatch_female_vert_6, symbol micromatch_female_TOP_ENTRY_locking_6
- added U1: RJ45_VT, footprints:RJ45-Vertical, symbol RJ45_VT
- J2: renamed from J?; footprint (none) -> footprints:Ampseal_14
Connections:
- net +12V: now also J1.1
- net AT_RESET: now also J1.7, U1.3 (RESET)
- net CANH: now also J1.9, U1.2 (CANH)
- net CANL: now also J1.8, U1.1 (CANL)
- net GND: now also J1.2, U1.11 (GND), U1.13 (GND), U1.14 (GND), U1.8 (GND), U1.9 (GND)
- net LED1: now also J1.10, U1.10 (LED_1)
- net LED2: now also J1.11, U1.12 (LED_2)
- net MISO: now also J1.5, U1.5 (MISO)
- net MOSI: now also J1.4, U1.6 (MOSI)
- net SCK: now also J1.6, U1.4 (SCK)
- net VCC: now also J1.3, U1.7 (5V)
- no-connect marks 0 -> 14
Changed lines of the file:
@@
 EESchema Schematic File Version 2
+LIBS:ExternalInterface-rescue
 LIBS:power
 LIBS:device
@@
 Comment4 ""
 $EndDescr
-$Comp
-L micromatch_female_RA_14 J?
-U 1 1 5A64D00C
-P 2160 1950
-F 0 "J?" H 2060 3150 60  0000 C CNN
-F 1 "micromatch_female_RA_14" H 2110 1600 60  0000 C CNN
-F 2 "footprints:micromatch_female_ra_14" H 1960 3050 60  0001 C CNN
-F 3 "" H 2060 3150 60  0001 C CNN
-F 4 "https://www.digikey.com/product-detail/en/te-connectivity-amp-connectors/1-338070-4/A99487CT-ND/1955789" H 2160 3250 60  0001 C CNN "PurchasingLink"
-F 5 "Digi-Key" H 2260 3350 60  0001 C CNN "MFN"
-F 6 "A99487CT-ND" H 2360 3450 60  0001 C CNN "MPN"
-F 7 "Value" H 2460 3550 60  0001 C CNN "Package"
-	1    2160 1950
-	-1   0    0    1
-$EndComp
 Text GLabel 2010 2050 0    60   Input ~ 0
 LED2
@@
 MOSI
 $Comp
-L VCC #PWR?
+L VCC #PWR01
 U 1 1 5A64D19F
 P 1960 2850
-F 0 "#PWR?" H 1960 2700 50  0001 C CNN
+F 0 "#PWR01" H 1960 2700 50  0001 C CNN
 F 1 "VCC" H 1960 3000 50  0000 C CNN
 F 2 "" H 1960 2850 50  0001 C CNN
@@
 $EndComp
 $Comp
-L GND #PWR?
+L GND #PWR02
 U 1 1 5A64D1B5
 P 1960 2950
-F 0 "#PWR?" H 1960 2700 50  0001 C CNN
+F 0 "#PWR02" H 1960 2700 50  0001 C CNN
 F 1 "GND" H 1960 2800 50  0000 C CNN
 F 2 "" H 1960 2950 50  0001 C CNN
@@
 $EndComp
 $Comp
-L +12V #PWR?
+L +12V #PWR03
 U 1 1 5A64D1CB
 P 1960 3050
-F 0 "#PWR?" H 1960 2900 50  0001 C CNN
+F 0 "#PWR03" H 1960 2900 50  0001 C CNN
 F 1 "+12V" H 1960 3190 50  0000 C CNN
 F 2 "" H 1960 3050 50  0001 C CNN
@@
 $EndComp
 $Comp
-L PWR_FLAG #FLG?
+L PWR_FLAG #FLG04
 U 1 1 5A64D1E1
 P 3550 1640
-F 0 "#FLG?" H 3550 1715 50  0001 C CNN
+F 0 "#FLG04" H 3550 1715 50  0001 C CNN
 F 1 "PWR_FLAG" H 3550 1790 50  0000 C CNN
 F 2 "" H 3550 1640 50  0001 C CNN
@@
 $EndComp
 $Comp
-L PWR_FLAG #FLG?
+L PWR_FLAG #FLG05
 U 1 1 5A64D1F8
 P 3800 1640
-F 0 "#FLG?" H 3800 1715 50  0001 C CNN
+F 0 "#FLG05" H 3800 1715 50  0001 C CNN
 F 1 "PWR_FLAG" H 3800 1790 50  0000 C CNN
 F 2 "" H 3800 1640 50  0001 C CNN
@@
 $EndComp
 $Comp
-L PWR_FLAG #FLG?
+L PWR_FLAG #FLG06
 U 1 1 5A64D206
 P 4030 1640
-F 0 "#FLG?" H 4030 1715 50  0001 C CNN
+F 0 "#FLG06" H 4030 1715 50  0001 C CNN
 F 1 "PWR_FLAG" H 4030 1790 50  0000 C CNN
 F 2 "" H 4030 1640 50  0001 C CNN
@@
 $EndComp
 $Comp
-L VCC #PWR?
+L VCC #PWR07
 U 1 1 5A64D214
 P 3550 1720
-F 0 "#PWR?" H 3550 1570 50  0001 C CNN
+F 0 "#PWR07" H 3550 1570 50  0001 C CNN
 F 1 "VCC" H 3550 1870 50  0000 C CNN
 F 2 "" H 3550 1720 50  0001 C CNN
@@
 $EndComp
 $Comp
-L GND #PWR?
+L GND #PWR08
 U 1 1 5A64D222
 P 3800 1730
-F 0 "#PWR?" H 3800 1480 50  0001 C CNN
+F 0 "#PWR08" H 3800 1480 50  0001 C CNN
 F 1 "GND" H 3800 1580 50  0000 C CNN
 F 2 "" H 3800 1730 50  0001 C CNN
@@
 $EndComp
 $Comp
-L +12V #PWR?
+L +12V #PWR09
 U 1 1 5A64D230
 P 4030 1720
-F 0 "#PWR?" H 4030 1570 50  0001 C CNN
+F 0 "#PWR09" H 4030 1570 50  0001 C CNN
 F 1 "+12V" H 4030 1860 50  0000 C CNN
 F 2 "" H 4030 1720 50  0001 C CNN
@@
 	-1   0    0    1
 $EndComp
-Wire Wire Line
-	2010 2950 1960 2950
-Wire Wire Line
-	2010 2850 1960 2850
-Wire Wire Line
-	2010 3050 1960 3050
-Wire Wire Line
-	3550 1640 3550 1720
-Wire Wire Line
-	3800 1640 3800 1730
-Wire Wire Line
-	4030 1640 4030 1720
-$Comp
-L Ampseal_14 J?
+$Comp
+L Ampseal_14 J2
 U 1 1 5A64D29C
 P 2180 4340
-F 0 "J?" H 1930 5090 60  0000 C CNN
+F 0 "J2" H 1930 5090 60  0000 C CNN
 F 1 "Ampseal_14" H 1880 3590 60  0000 L CNN
-F 2 "" H 1980 4640 60  0001 C CNN
+F 2 "footprints:Ampseal_14" H 1980 4640 60  0001 C CNN
 F 3 "" H 1980 4640 60  0001 C CNN
 	1    2180 4340
@@
 $EndComp
 $Comp
-L +12V #PWR?
+L +12V #PWR010
 U 1 1 5A66322D
 P 1910 4190
-F 0 "#PWR?" H 1910 4040 50  0001 C CNN
+F 0 "#PWR010" H 1910 4040 50  0001 C CNN
 F 1 "+12V" H 1910 4330 50  0000 C CNN
 F 2 "" H 1910 4190 50  0001 C CNN
@@
 $EndComp
 $Comp
-L +12V #PWR?
+L +12V #PWR011
 U 1 1 5A66323E
 P 1910 3790
-F 0 "#PWR?" H 1910 3640 50  0001 C CNN
+F 0 "#PWR011" H 1910 3640 50  0001 C CNN
 F 1 "+12V" H 1910 3930 50  0000 C CNN
 F 2 "" H 1910 3790 50  0001 C CNN
@@
 CANL
 $Comp
-L GND #PWR?
+L GND #PWR012
 U 1 1 5A663271
 P 1900 4590
-F 0 "#PWR?" H 1900 4340 50  0001 C CNN
+F 0 "#PWR012" H 1900 4340 50  0001 C CNN
 F 1 "GND" H 1900 4440 50  0000 C CNN
 F 2 "" H 1900 4590 50  0001 C CNN
@@
 $EndComp
 $Comp
-L GND #PWR?
+L GND #PWR013
 U 1 1 5A663282
 P 1910 3690
-F 0 "#PWR?" H 1910 3440 50  0001 C CNN
+F 0 "#PWR013" H 1910 3440 50  0001 C CNN
 F 1 "GND" H 1910 3540 50  0000 C CNN
 F 2 "" H 1910 3690 50  0001 C CNN
@@
 $EndComp
 $Comp
-L GND #PWR?
+L GND #PWR014
 U 1 1 5A663293
 P 1910 3890
-F 0 "#PWR?" H 1910 3640 50  0001 C CNN
+F 0 "#PWR014" H 1910 3640 50  0001 C CNN
 F 1 "GND" H 1910 3740 50  0000 C CNN
 F 2 "" H 1910 3890 50  0001 C CNN
@@
 	0    1    1    0
 $EndComp
+$Comp
+L RJ45_VT U1
+U 1 1 5A7B523B
+P 3600 3230
+F 0 "U1" H 3600 2640 60  0000 C CNN
+F 1 "RJ45_VT" H 3610 3890 60  0000 C CNN
+F 2 "footprints:RJ45-Vertical" H 3500 2540 60  0001 C CNN
+F 3 "" H 3600 2640 60  0001 C CNN
+	1    3600 3230
+	1    0    0    -1
+$EndComp
+Wire Wire Line
+	2010 2950 1960 2950
+Wire Wire Line
+	2010 2850 1960 2850
+Wire Wire Line
+	2010 3050 1960 3050
+Wire Wire Line
+	3550 1640 3550 1720
+Wire Wire Line
+	3800 1640 3800 1730
+Wire Wire Line
+	4030 1640 4030 1720
 Wire Wire Line
 	1910 3690 1980 3690
@@
 Wire Wire Line
 	1900 4590 1980 4590
+Text GLabel 4450 2800 2    60   Input ~ 0
+MISO
+Text GLabel 4450 2900 2    60   Input ~ 0
+MOSI
+Text GLabel 3530 3620 3    60   Input ~ 0
+LED1
+Text GLabel 3810 3620 3    60   Input ~ 0
+LED2
+Text GLabel 3120 3100 0    60   Input ~ 0
+SCK
+Text GLabel 3120 3000 0    60   Input ~ 0
+AT_RESET
+Text GLabel 3120 2900 0    60   Input ~ 0
+CANH
+Text GLabel 3120 2800 0    60   Input ~ 0
+CANL
+$Comp
+L GND #PWR015
+U 1 1 5A7B530F
+P 4110 4050
+F 0 "#PWR015" H 4110 3800 50  0001 C CNN
+F 1 "GND" H 4110 3900 50  0000 C CNN
+F 2 "" H 4110 4050 50  0001 C CNN
+F 3 "" H 4110 4050 50  0001 C CNN
+	1    4110 4050
+	1    0    0    -1
+$EndComp
+Wire Wire Line
+	4110 4050 4110 3620
+Wire Wire Line
+	4000 3620 4000 3980
+Wire Wire Line
+	3420 3980 4450 3980
+Connection ~ 4110 3980
+Wire Wire Line
+	3700 3620 3700 3980
+Connection ~ 4000 3980
+Wire Wire Line
+	3420 3620 3420 3980
+Connection ~ 3700 3980
+Wire Wire Line
+	4450 3980 4450 3100
+$Comp
+L VCC #PWR016
+U 1 1 5A7B538A
+P 4790 3000
+F 0 "#PWR016" H 4790 2850 50  0001 C CNN
+F 1 "VCC" H 4790 3150 50  0000 C CNN
+F 2 "" H 4790 3000 50  0001 C CNN
+F 3 "" H 4790 3000 50  0001 C CNN
+	1    4790 3000
+	1    0    0    -1
+$EndComp
+Wire Wire Line
+	4450 3000 4790 3000
+NoConn ~ 2010 1750
+NoConn ~ 2010 1850
+NoConn ~ 2010 1950
+NoConn ~ 1980 3990
+NoConn ~ 1980 4090
+NoConn ~ 1980 4490
+NoConn ~ 1980 4890
+NoConn ~ 1980 4990
+$Comp
+L micromatch_female_TOP_ENTRY_locking_14 J1
+U 1 1 5A7B7983
+P 2310 2400
+F 0 "J1" H 2360 3150 60  0000 C CNN
+F 1 "micromatch_female_TOP_ENTRY_locking_14" H 2410 1600 60  0000 C CNN
+F 2 "footprints:micromatch_female_vert_14" H 2260 3050 60  0001 C CNN
+F 3 "" H 2360 3150 60  0001 C CNN
+F 4 "https://www.digikey.com/product-detail/en/te-connectivity-amp-connectors/1-338068-4/A99502CT-ND/1955735" H 2310 3700 60  0001 C CNN "PurchasingLink"
+F 5 "Digi-Key" H 2410 3800 60  0001 C CNN "MFN"
+F 6 "A99502CT-ND" H 2510 3900 60  0001 C CNN "MPN"
+F 7 "Value" H 2610 4000 60  0001 C CNN "Package"
+	1    2310 2400
+	-1   0    0    1
+$EndComp
+$Comp
+L micromatch_female_TOP_ENTRY_locking_6 J3
+U 1 1 5A7B962C
+P 4670 1580
+F 0 "J3" H 4670 1930 60  0000 C CNN
+F 1 "micromatch_female_TOP_ENTRY_locking_6" H 4770 1180 60  0000 C CNN
+F 2 "footprints:micromatch_female_vert_6" H 4570 1830 60  0001 C CNN
+F 3 "" H 4670 1930 60  0001 C CNN
+F 4 "https://www.digikey.com/product-detail/en/te-connectivity-amp-connectors/338068-6/A99437CT-ND/1955739" H 4670 2880 60  0001 C CNN "PurchasingLink"
+F 5 "Digi-Key" H 4770 2980 60  0001 C CNN "MFN"
+F 6 "A99437CT-ND" H 4870 3080 60  0001 C CNN "MPN"
+F 7 "Value" H 4970 3180 60  0001 C CNN "Package"
+	1    4670 1580
+	0    1    1    0
+$EndComp
+NoConn ~ 4920 1830
+NoConn ~ 4820 1830
+NoConn ~ 4720 1830
+NoConn ~ 4620 1830
+NoConn ~ 4520 1830
+NoConn ~ 4420 1830
 $EndSCHEMATC

Commit message: Gerbers and PDFs
Connections:
- net +12V: now also J2.12, J2.8; no longer J2.13, J2.9
- net CANH: now also J2.10, J2.6; no longer J2.4, J2.8
- net CANL: now also J2.11; no longer J2.3
- net GND: now also J2.1, J2.2, J2.3; no longer J2.12, J2.14, J2.5
- no-connect marks 14 -> 18
Changed lines of the file:
@@
 $Comp
 L +12V #PWR010
-U 1 1 5A66322D
-P 1910 4190
-F 0 "#PWR010" H 1910 4040 50  0001 C CNN
-F 1 "+12V" H 1910 4330 50  0000 C CNN
-F 2 "" H 1910 4190 50  0001 C CNN
-F 3 "" H 1910 4190 50  0001 C CNN
-	1    1910 4190
+U 1 1 5A66323E
+P 1980 4290
+F 0 "#PWR010" H 1980 4140 50  0001 C CNN
+F 1 "+12V" H 1980 4430 50  0000 C CNN
+F 2 "" H 1980 4290 50  0001 C CNN
+F 3 "" H 1980 4290 50  0001 C CNN
+	1    1980 4290
 	0    -1   -1   0
 $EndComp
-$Comp
-L +12V #PWR011
-U 1 1 5A66323E
-P 1910 3790
-F 0 "#PWR011" H 1910 3640 50  0001 C CNN
-F 1 "+12V" H 1910 3930 50  0000 C CNN
-F 2 "" H 1910 3790 50  0001 C CNN
-F 3 "" H 1910 3790 50  0001 C CNN
-	1    1910 3790
-	0    -1   -1   0
-$EndComp
-Text GLabel 1980 4690 0    60   Input ~ 0
+Text GLabel 1980 4090 0    60   Input ~ 0
 CANH
-Text GLabel 1980 4290 0    60   Input ~ 0
+Text GLabel 1980 4490 0    60   Input ~ 0
 CANH
-Text GLabel 1980 4790 0    60   Input ~ 0
+Text GLabel 1980 3990 0    60   Input ~ 0
 CANL
 Text GLabel 1980 4390 0    60   Input ~ 0
 CANL
 $Comp
-L GND #PWR012
-U 1 1 5A663271
-P 1900 4590
-F 0 "#PWR012" H 1900 4340 50  0001 C CNN
-F 1 "GND" H 1900 4440 50  0000 C CNN
-F 2 "" H 1900 4590 50  0001 C CNN
-F 3 "" H 1900 4590 50  0001 C CNN
-	1    1900 4590
+L GND #PWR011
+U 1 1 5A663282
+P 1910 4790
+F 0 "#PWR011" H 1910 4540 50  0001 C CNN
+F 1 "GND" H 1910 4640 50  0000 C CNN
+F 2 "" H 1910 4790 50  0001 C CNN
+F 3 "" H 1910 4790 50  0001 C CNN
+	1    1910 4790
 	0    1    1    0
 $EndComp
 $Comp
-L GND #PWR013
-U 1 1 5A663282
-P 1910 3690
-F 0 "#PWR013" H 1910 3440 50  0001 C CNN
-F 1 "GND" H 1910 3540 50  0000 C CNN
-F 2 "" H 1910 3690 50  0001 C CNN
-F 3 "" H 1910 3690 50  0001 C CNN
-	1    1910 3690
-	0    1    1    0
-$EndComp
-$Comp
-L GND #PWR014
+L GND #PWR012
 U 1 1 5A663293
-P 1910 3890
-F 0 "#PWR014" H 1910 3640 50  0001 C CNN
-F 1 "GND" H 1910 3740 50  0000 C CNN
-F 2 "" H 1910 3890 50  0001 C CNN
-F 3 "" H 1910 3890 50  0001 C CNN
-	1    1910 3890
+P 1910 4990
+F 0 "#PWR012" H 1910 4740 50  0001 C CNN
+F 1 "GND" H 1910 4840 50  0000 C CNN
+F 2 "" H 1910 4990 50  0001 C CNN
+F 3 "" H 1910 4990 50  0001 C CNN
+	1    1910 4990
 	0    1    1    0
 $EndComp
@@
 	4030 1640 4030 1720
 Wire Wire Line
-	1910 3690 1980 3690
+	1910 4790 1980 4790
 Wire Wire Line
-	1910 3790 1980 3790
+	1910 4890 1980 4890
 Wire Wire Line
-	1910 3890 1980 3890
-Wire Wire Line
-	1910 4190 1980 4190
-Wire Wire Line
-	1900 4590 1980 4590
+	1910 4990 1980 4990
 Text GLabel 4450 2800 2    60   Input ~ 0
 MISO
@@
 CANL
 $Comp
-L GND #PWR015
+L GND #PWR013
 U 1 1 5A7B530F
 P 4110 4050
-F 0 "#PWR015" H 4110 3800 50  0001 C CNN
+F 0 "#PWR013" H 4110 3800 50  0001 C CNN
 F 1 "GND" H 4110 3900 50  0000 C CNN
 F 2 "" H 4110 4050 50  0001 C CNN
@@
 	4450 3980 4450 3100
 $Comp
-L VCC #PWR016
+L VCC #PWR014
 U 1 1 5A7B538A
 P 4790 3000
-F 0 "#PWR016" H 4790 2850 50  0001 C CNN
+F 0 "#PWR014" H 4790 2850 50  0001 C CNN
 F 1 "VCC" H 4790 3150 50  0000 C CNN
 F 2 "" H 4790 3000 50  0001 C CNN
@@
 NoConn ~ 2010 1850
 NoConn ~ 2010 1950
-NoConn ~ 1980 3990
-NoConn ~ 1980 4090
-NoConn ~ 1980 4490
-NoConn ~ 1980 4890
-NoConn ~ 1980 4990
 $Comp
 L micromatch_female_TOP_ENTRY_locking_14 J1
@@
 NoConn ~ 4520 1830
 NoConn ~ 4420 1830
+$Comp
+L GND #PWR015
+U 1 1 5A8B7071
+P 1910 4890
+F 0 "#PWR015" H 1910 4640 50  0001 C CNN
+F 1 "GND" H 1910 4740 50  0000 C CNN
+F 2 "" H 1910 4890 50  0001 C CNN
+F 3 "" H 1910 4890 50  0001 C CNN
+	1    1910 4890
+	0    1    1    0
+$EndComp
+$Comp
+L +12V #PWR016
+U 1 1 5A8B721D
+P 1980 3890
+F 0 "#PWR016" H 1980 3740 50  0001 C CNN
+F 1 "+12V" H 1980 4030 50  0000 C CNN
+F 2 "" H 1980 3890 50  0001 C CNN
+F 3 "" H 1980 3890 50  0001 C CNN
+	1    1980 3890
+	0    -1   -1   0
+$EndComp
+NoConn ~ 1980 3790
+NoConn ~ 1980 3690
+NoConn ~ 1980 4190
+NoConn ~ 1980 4690
+NoConn ~ 1980 4590
+NoConn ~ 3450 2505
+NoConn ~ 215  5860
+NoConn ~ 760  3810
+NoConn ~ 4515 1515
 $EndSCHEMATC
