File: boards/TSAL/TSAL v2/TSAL v2.sch (KiCad schematic (older format))
At the start: 26 parts, among them J1 Ultrafit_2, J2 Ultrafit_2, J3 micromatch_female_TOP_ENTRY_l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, Q1 NMOS_GSD_30V, U1 LR8K4-G, U2 ZXRE160, U3 MCP6001RT, U4 LTV-356T

Commit message: Updated the purchasing links
Parts:
- R7: Webpage https://www.digikey.com/product-detail/en/panasonic-electronic-components/ERA-6AEB1783V/P178KDATR-ND/2025864 -> https://www.digikey.com/product-detail/en/panasonic-electronic-components/ERA-6AEB1783V/P178KDACT-ND/3074993
- U2: Webpage https://www.digikey.com/product-detail/en/diodes-incorporated/ZXRE160H5TA/ZXRE160H5TADICT-ND/3677932 -> https://www.digikey.com/product-detail/en/diodes-incorporated/ZXRE160AET5TA/ZXRE160AET5TADICT-ND/3677927
Changed lines of the file:
@@
 F 4 "DigiKey" H 7000 5150 60  0001 C CNN "MFN"
 F 5 "ZXRE160FT4-7DICT-ND" H 7100 5250 60  0001 C CNN "MPN"
-F 6 "https://www.digikey.com/product-detail/en/diodes-incorporated/ZXRE160H5TA/ZXRE160H5TADICT-ND/3677932" H 7200 5350 60  0001 C CNN "Webpage"
+F 6 "https://www.digikey.com/product-detail/en/diodes-incorporated/ZXRE160AET5TA/ZXRE160AET5TADICT-ND/3677927" H 7200 5350 60  0001 C CNN "Webpage"
 	1    6900 5650
 	0    1    1    0
@@
 F 4 "Digikey" V 7480 2650 60  0001 C CNN "MFN"
 F 5 "P178KDATR-ND" V 7580 2750 60  0001 C CNN "MPN"
-F 6 "https://www.digikey.com/product-detail/en/panasonic-electronic-components/ERA-6AEB1783V/P178KDATR-ND/2025864" V 7680 2850 60  0001 C CNN "Webpage"
+F 6 "https://www.digikey.com/product-detail/en/panasonic-electronic-components/ERA-6AEB1783V/P178KDACT-ND/3074993" V 7680 2850 60  0001 C CNN "Webpage"
 	1    7300 2550
 	0    1    1    0
