File: boards/Precharge/Precharge_Schematics.sch (KiCad schematic (older format))
At the start: 5 parts, among them J1 Ultrafit_2, J2 Ultrafit_2, J3 Ultrafit_2, K1 G2RL-1-E

Commit message: Updated Layout
Parts:
- J1: value Ultrafit_2 -> BAT+
- J2: value Ultrafit_2 -> Shutdown_LSD
- J3: value Ultrafit_2 -> TS+
Changed lines of the file:
@@
 EESchema Schematic File Version 2
-LIBS:AIL_Precharge_Schematics-rescue
 LIBS:power
 LIBS:device
@@
 LIBS:valves
 LIBS:formula
-LIBS:AIL_Precharge_Schematics-cache
 EELAYER 25 0
 EELAYER END
@@
 NoConn ~ 2150 1100
 NoConn ~ 2350 3100
-Text Label 1100 4300 0    60   ~ 0
-TS
-Text Label 1500 1100 0    60   ~ 0
-BAT+
 $Comp
 L Ultrafit_2 J1
@@
 P 1900 1050
 F 0 "J1" H 1900 1200 60  0000 C CNN
-F 1 "Ultrafit_2" H 2000 850 60  0000 C CNN
+F 1 "BAT+" H 2000 850 60  0000 C CNN
 F 2 "footprints:Ultrafit_2" H 1800 1100 60  0001 C CNN
 F 3 "" H 1900 1200 60  0001 C CNN
@@
 U 1 1 59F29554
 P 1400 3600
-F 0 "J2" H 1150 3600 60  0000 C CNN
-F 1 "Ultrafit_2" H 1500 3400 60  0000 C CNN
+F 0 "J2" H 1400 3800 60  0000 C CNN
+F 1 "Shutdown_LSD" H 1500 3400 60  0000 C CNN
 F 2 "footprints:Ultrafit_2" H 1300 3650 60  0001 C CNN
 F 3 "" H 1400 3750 60  0001 C CNN
@@
 P 1400 4300
 F 0 "J3" H 1400 4450 60  0000 C CNN
-F 1 "Ultrafit_2" H 1500 4100 60  0000 C CNN
+F 1 "TS+" H 1500 4100 60  0000 C CNN
 F 2 "footprints:Ultrafit_2" H 1300 4350 60  0001 C CNN
 F 3 "" H 1400 4450 60  0001 C CNN
@@
 Text GLabel 2850 3100 3    60   Input ~ 0
 Low_Side_Drive
-Text Label 1050 3850 0    60   ~ 0
-ShutDown_LowSideDrive
 $Comp
 L R_1k_HS R1
